Commit message: added side bogies, but it is still a work in progress

File: urdf/rover_dummy.xacro (robot description, xacro)
@@ -8,4 +8,5 @@
   <!-- Warning: the wheel_radius value must be the same as in the YAML configuration file-->
   <xacro:property name="wheel_radius" value="${size_link / 2}" />
+  <xacro:property name="variant" value="1.0" />
   <xacro:property name="limit_drive_effort" value="100.0" />
   <xacro:property name="limit_drive_velocity" value="1.0" />
@@ -14,4 +15,6 @@
   <xacro:property name="limit_steer_upper" value="${pi / 2}" />
   <xacro:property name="limit_steer_velocity" value="1.0" />
+  <xacro:property name="side_boogie_lower" value="${-pi / 2}" />
+  <xacro:property name="side_boogie_upper" value="${pi / 2}" />
   <!-- Import all Gazebo-customization elements, including Gazebo colors and plugins -->
   <xacro:include filename="$(find rover_config)/urdf/rover_dummy.gazebo" />
@@ -41,12 +44,46 @@
     </visual>
   </link>
+  <!-- Definition for a side boogie assembly -->
+  <xacro:macro name="side_boogie" params="position *origin_boogie">
+    <xacro:property name="boogie_link" value="link_boogie_${position}" />
+    <joint name="joint_boogie_${position}" type="fixed">
+      <parent link="base_link"/>
+      <child link="link_boogie_${position}"/>
+      <xacro:insert_block name="origin_boogie" />
+      <limit effort="0" lower="${side_boogie_lower}" upper="${side_boogie_upper}" velocity="0"/>
+      <axis xyz="0 1 0"/>
+    </joint>
+    <link name="link_boogie_${position}">
+      <collision>
+        <geometry>
+          <cylinder length="0.3" radius="0.05"/>
+        </geometry>
+      </collision>
+      <inertial>
+        <mass value="${mass}"/>
+        <inertia
+              ixx="${mass / 12.0 * (size_link * size_link / 2)}"
+              iyy="${mass / 12.0 * (size_link * size_link / 2)}"
+              izz="${mass / 12.0 * (size_link * size_link / 2)}"
+              ixy="0"
+              ixz="0"
+              iyz="0"/>
+      </inertial>
+      <visual>
+        <origin xyz="0 0 0" rpy="0 0 0"/>
+        <geometry>
+          <cylinder length="0.3" radius="0.05"/>
+        </geometry>
+      </visual>
+    </link>
+  </xacro:macro>
   <!-- Definition for a wheel assembly -->
-  <xacro:macro name="wheel_assembly" params="position *origin_DEP">
+  <xacro:macro name="wheel_assembly" params="position variant boogie_name *origin_DEP">
     <joint name="joint_DEP_${position}" type="fixed">
-      <parent link="base_link"/>
+      <parent link="link_boogie_${boogie_name}"/>
       <child link="link_DEP_${position}"/>
       <limit effort="${limit_steer_effort}" lower="${limit_steer_lower}" upper="${limit_steer_upper}" velocity="${limit_steer_velocity}"/>
       <xacro:insert_block name="origin_DEP" />
-      <axis xyz="0 1 0"/>
+      <axis xyz="0 0 1"/>
       <dynamics damping="${damping}" friction="${friction}"/>
     </joint>
@@ -117,5 +154,5 @@
     <link name="link_DRV_${position}">
       <collision>
-        <origin xyz="0 0 0" rpy="${pi / 2} 0 0"/>
+        <origin xyz="0 0 0" rpy="0 0 0"/>
         <geometry>
           <cylinder length="${size_link}" radius="${wheel_radius}"/>
@@ -133,5 +170,5 @@
       </inertial>
       <visual>
-        <origin xyz="0 0 0" rpy="${pi / 2} 0 0"/>
+        <origin xyz="0 0 0" rpy="0 0 0"/>
         <geometry>
           <cylinder length="${size_link}" radius="${wheel_radius}"/>
@@ -159,22 +196,13 @@
   </xacro:macro>
   <!-- Define all the wheel assemblies as set their positions -->
-  <xacro:wheel_assembly position="RF">
-    <origin xyz="${(size_base / 2 + size_link)} ${-(size_base / 2 + size_link)} 0" rpy="0 0 0"/>
+  <xacro:property name="boogie_name" value="L" />
+  <xacro:side_boogie position="${boogie_name}">
+    <origin xyz="0 0 0" rpy="1.57 0 0"/>
+  </xacro:side_boogie>
+  <xacro:wheel_assembly position="RR" variant="1.0" boogie_name="${boogie_name}">
+    <origin xyz="0 0 0" rpy="1.57 0 0"/>
   </xacro:wheel_assembly>
-  <xacro:wheel_assembly position="RM">
-    <origin xyz="0 ${-(size_base / 2 + size_link)} 0" rpy="0 0 0"/>
-  </xacro:wheel_assembly>
-  <xacro:wheel_assembly position="RR">
-    <!-- <origin xyz="${-(size_base / 2 + size_link)} ${-(size_base / 2 + size_link)} 0" rpy="0 0 0"/> -->
-    <origin xyz="${-(size_base / 2 + size_link)} ${-(size_base / 2 + size_link)} 0" rpy="1.57 0 0"/>
-  </xacro:wheel_assembly>
-  <xacro:wheel_assembly position="LF">
-    <origin xyz="${(size_base / 2 + size_link)} ${(size_base / 2 + size_link)} 0" rpy="0 0 0"/>
-  </xacro:wheel_assembly>
-  <xacro:wheel_assembly position="LM">
-    <origin xyz="0 ${(size_base / 2 + size_link)} 0" rpy="0 0 0"/>
-  </xacro:wheel_assembly>
-  <xacro:wheel_assembly position="LR">
-    <origin xyz="${-(size_base / 2 + size_link)} ${(size_base / 2 + size_link)} 0" rpy="1.57 0 0"/>
+  <xacro:wheel_assembly position="RM" variant="1.0" boogie_name="${boogie_name}">
+    <origin xyz="0 0 0" rpy="1.57 0 0"/>
   </xacro:wheel_assembly>
 </robot>
