Commit message: added main marta dims

File: urdf/exoter.xacro (robot description, xacro)
@@ -6,6 +6,5 @@
   <xacro:property name="size_base" value="0.5" />
   <xacro:property name="size_link" value="0.15" />
-  <!-- Warning: the wheel_radius value must be the same as in the YAML configuration file-->
-  <xacro:property name="wheel_radius" value="0.08" />
+  <xacro:property name="wheel_radius" value="${0.1425 / 2}" />
   <xacro:property name="variant" value="1.0" />
   <xacro:property name="limit_drive_effort" value="100.0" />
@@ -15,6 +14,6 @@
   <xacro:property name="limit_steer_upper" value="${pi / 2}" />
   <xacro:property name="limit_steer_velocity" value="1.0" />
-  <xacro:property name="side_boogie_lower" value="${-pi / 4}" />
-  <xacro:property name="side_boogie_upper" value="${pi / 4}" />
+  <xacro:property name="side_bogie_lower" value="${-pi / 4}" />
+  <xacro:property name="side_bogie_upper" value="${pi / 4}" />
   <!-- Import all Gazebo-customization elements, including Gazebo colors and plugins -->
   <xacro:include filename="$(find rover_config)/urdf/marta.gazebo" />
@@ -44,15 +43,15 @@
     </visual>
   </link>
-  <!-- Definition for a side boogie assembly -->
-  <xacro:macro name="boogie" params="position *origin_boogie">
-    <xacro:property name="boogie_link" value="link_boogie_${position}" />
-    <joint name="joint_boogie_${position}" type="revolute">
+  <!-- Definition for a side bogie assembly -->
+  <xacro:macro name="bogie" params="position *origin_bogie">
+    <xacro:property name="bogie_link" value="link_bogie_${position}" />
+    <joint name="joint_bogie_${position}" type="revolute">
       <parent link="base_link"/>
-      <child link="link_boogie_${position}"/>
-      <xacro:insert_block name="origin_boogie" />
-      <limit effort="0" lower="${side_boogie_lower}" upper="${side_boogie_upper}" velocity="0"/>
+      <child link="link_bogie_${position}"/>
+      <xacro:insert_block name="origin_bogie" />
+      <limit effort="0" lower="${side_bogie_lower}" upper="${side_bogie_upper}" velocity="0"/>
       <axis xyz="0 0 1"/>
     </joint>
-    <link name="link_boogie_${position}">
+    <link name="link_bogie_${position}">
       <collision>
         <origin xyz="0 0 0.03" rpy="0 ${pi / 2} 0"/>
@@ -81,7 +80,7 @@
   <!-- Definition for a wheel assembly -->
   <!-- Driving direction is used to invert the direction of the deployment and driving joint -->
-  <xacro:macro name="wheel_assembly" params="position boogie_name driving_direction str_type:=revolute *origin_DEP *origin_STR">
+  <xacro:macro name="wheel_assembly" params="position bogie_name driving_direction str_type:=revolute *origin_DEP *origin_STR">
     <joint name="joint_DEP_${position}" type="revolute">
-      <parent link="link_boogie_${boogie_name}"/>
+      <parent link="link_bogie_${bogie_name}"/>
       <child link="link_DEP_${position}"/>
       <limit effort="${limit_steer_effort}" lower="${limit_steer_lower}" upper="${limit_steer_upper}" velocity="${limit_steer_velocity}"/>
@@ -200,39 +199,39 @@
   <!-- Define all the wheel assemblies & bogies. Set their positions -->
   <!-- LEFT BOGIE  -->
-  <xacro:property name="side_boogie_left_name" value="LFB" />
-  <xacro:boogie position="${side_boogie_left_name}">
+  <xacro:property name="side_bogie_left_name" value="LFB" />
+  <xacro:bogie position="${side_bogie_left_name}">
     <origin xyz="0.3 ${size_base / 2} 0" rpy="${- pi / 2} 0 0"/>
-  </xacro:boogie>
-  <xacro:wheel_assembly position="LF" boogie_name="${side_boogie_left_name}" driving_direction="1">
+  </xacro:bogie>
+  <xacro:wheel_assembly position="LF" bogie_name="${side_bogie_left_name}" driving_direction="1">
     <origin xyz="0.2 0 0.05" rpy="0 0 0"/>
     <origin xyz="0.1 0 0.1" rpy="${pi / 2} 0 0"/>
   </xacro:wheel_assembly>
-  <xacro:wheel_assembly position="LM" boogie_name="${side_boogie_left_name}" driving_direction="1" str_type="fixed">
+  <xacro:wheel_assembly position="LM" bogie_name="${side_bogie_left_name}" driving_direction="1" str_type="fixed">
     <origin xyz="-0.2 0 0.05" rpy="0 0 0"/>
     <origin xyz="-0.1 0 0.1" rpy="${pi / 2} 0 0"/>
   </xacro:wheel_assembly>
   <!-- RIGHT BOGIE  -->
-  <xacro:property name="side_boogie_right_name" value="RFB" />
-  <xacro:boogie position="${side_boogie_right_name}">
+  <xacro:property name="side_bogie_right_name" value="RFB" />
+  <xacro:bogie position="${side_bogie_right_name}">
     <origin xyz="0.3 -${size_base / 2} 0" rpy="${- pi / 2} 0 ${pi}"/>
-  </xacro:boogie>
-  <xacro:wheel_assembly position="RF" boogie_name="${side_boogie_right_name}" driving_direction="-1">
+  </xacro:bogie>
+  <xacro:wheel_assembly position="RF" bogie_name="${side_bogie_right_name}" driving_direction="-1">
     <origin xyz="-0.2 0 0.05" rpy="0 0 0"/>
     <origin xyz="-0.1 0 0.1" rpy="${pi / 2} 0 0"/>
   </xacro:wheel_assembly>
-  <xacro:wheel_assembly position="RM" boogie_name="${side_boogie_right_name}" driving_direction="-1" str_type="fixed">
+  <xacro:wheel_assembly position="RM" bogie_name="${side_bogie_right_name}" driving_direction="-1" str_type="fixed">
     <origin xyz="0.2 0 0.05" rpy="0 0 0"/>
     <origin xyz="0.1 0 0.1" rpy="${pi / 2} 0 0"/>
   </xacro:wheel_assembly>
   <!-- REAR BOGIE  -->
-  <xacro:property name="side_boogie_rear_name" value="MRB" />
-  <xacro:boogie position="${side_boogie_rear_name}">
+  <xacro:property name="side_bogie_rear_name" value="MRB" />
+  <xacro:bogie position="${side_bogie_rear_name}">
     <origin xyz="-${size_base / 2 + 0.05} 0 0" rpy="${- pi / 2} 0 ${pi / 2}"/>
-  </xacro:boogie>
-  <xacro:wheel_assembly position="LR" boogie_name="${side_boogie_rear_name}" driving_direction="1">
+  </xacro:bogie>
+  <xacro:wheel_assembly position="LR" bogie_name="${side_bogie_rear_name}" driving_direction="1">
     <origin xyz="0.3 0 0.05" rpy="0 ${pi / 2} 0"/>
     <origin xyz="-0.1 0 0.1" rpy="${pi / 2} 0 0"/>
   </xacro:wheel_assembly>
-  <xacro:wheel_assembly position="RR" boogie_name="${side_boogie_rear_name}" driving_direction="-1">
+  <xacro:wheel_assembly position="RR" bogie_name="${side_bogie_rear_name}" driving_direction="-1">
     <origin xyz="-0.3 0 0.05" rpy="0 ${3 * pi / 2} 0"/>
     <origin xyz="0.1 0 0.1" rpy="${pi / 2} 0 0"/>
