Commit message: Change name of link

File: urdf/lidar.xacro (robot description, xacro)
@@ -5,8 +5,8 @@
     <joint name="joint_lidar" type="fixed">
         <parent link="${parent_link}"/>
-        <child link="lidar_link"/>
+        <child link="link_lidar"/>
         <xacro:insert_block name="origin" />
     </joint>
-    <link name="lidar_link">
+    <link name="link_lidar">
         <visual>
         <origin xyz="0 0 0" rpy="0 0 0"/>

Commit message: Fixed Indent to be 2 spaces

File: urdf/lidar.xacro (robot description, xacro)
@@ -4,15 +4,15 @@
     <xacro:include filename="$(find rover_config)/urdf/lidar.gazebo" />
     <joint name="joint_lidar" type="fixed">
-        <parent link="${parent_link}"/>
-        <child link="link_lidar"/>
-        <xacro:insert_block name="origin" />
+      <parent link="${parent_link}"/>
+      <child link="link_lidar"/>
+      <xacro:insert_block name="origin" />
     </joint>
     <link name="link_lidar">
-        <visual>
+      <visual>
         <origin xyz="0 0 0" rpy="0 0 0"/>
         <geometry>
-            <box size="0.1 0.1 0.1"/>
+          <box size="0.1 0.1 0.1"/>
         </geometry>
-        </visual>
+      </visual>
     </link>
   </xacro:macro>
