Commit message: added PTU links and joints with STR in name so it works w/ the plugin

File: urdf/ptu.xacro (robot description, xacro)
@@ -2,7 +2,11 @@
 <robot xmlns:xacro="http://wiki.ros.org/xacro">
   <xacro:macro name="ptu" params="parent_link *origin">
+    <!-- PHYSICS -->
+    <xacro:property name="ptu_damping" value="2" />
+    <xacro:property name="ptu_friction" value="0.1" />
+    <xacro:include filename="$(find rover_config)/urdf/ptu.gazebo" />
     <!-- PARAMETERS -->
     <!-- MAST LINK -->
-    <xacro:property name="mast_r" value="0.022" />
+    <xacro:property name="mast_r" value="0.011" />
     <xacro:property name="mast_l" value="0.6375" />
     <xacro:property name="mast_mass" value="4.0" />
@@ -10,25 +14,34 @@
     <xacro:property name="pan_lower" value="-1.57" />
     <xacro:property name="pan_upper" value="1.57" />
-    <xacro:property name="joint_pan_z" value="${mast_l}" />
+    <xacro:property name="joint_pan_pos_z" value="${mast_l}" />
     <!-- PAN LINK -->
     <xacro:property name="link_pan_mass" value="0.1" />
-    <xacro:property name="link_pan_x" value="0.0" />
-    <xacro:property name="link_pan_y" value="0.0" />
-    <xacro:property name="link_pan_z" value="0.04" />
-    <xacro:property name="link_pan_pos_x" value="0.0" />
+    <xacro:property name="link_pan_x" value="0.05" />
+    <xacro:property name="link_pan_y" value="0.025" />
+    <xacro:property name="link_pan_z" value="0.025" />
+    <xacro:property name="link_pan_pos_x" value="-0.0125" />
     <xacro:property name="link_pan_pos_y" value="0.0" />
-    <xacro:property name="link_pan_pos_z" value="${link_pan_z}" />
+    <xacro:property name="link_pan_pos_z" value="${link_pan_z/2}" />
     <!-- TILT JOINT -->
     <xacro:property name="tilt_lower" value="-1.57" />
     <xacro:property name="tilt_upper" value="1.57" />
-    <xacro:property name="joint_tilt_z" value="${mast_l}" />
+    <xacro:property name="joint_tilt_pos_z" value="0.0265" />
+    <xacro:property name="joint_tilt_rot_x" value="${pi/2}" />
+    <!-- PAN LINK -->
+    <xacro:property name="link_tilt_mass" value="0.1" />
+    <xacro:property name="link_tilt_x" value="0.022" />
+    <xacro:property name="link_tilt_y" value="0.0035" />
+    <xacro:property name="link_tilt_z" value="0.072" />
+    <xacro:property name="link_tilt_pos_x" value="0.0" />
+    <xacro:property name="link_tilt_pos_y" value="0.01625" />
+    <xacro:property name="link_tilt_pos_z" value="0.0" />
     <!-- MAST JOINT -->
     <joint name="ptu_base" type="fixed">
       <parent link="${parent_link}"/>
-      <child link="mast"/>
+      <child link="link_mast"/>
       <xacro:insert_block name="origin" />
     </joint>
     <!-- MAST LINK -->
-    <link name="mast">
+    <link name="link_mast">
       <inertial>
         <mass value="${mast_mass}"/>
@@ -55,10 +68,11 @@
     </link>
     <!-- PAN JOINT -->
-    <joint name="pan" type="revolute">
-      <parent link="mast"/>
+    <joint name="joint_STR_pan" type="revolute">
+      <parent link="link_mast"/>
       <child link="link_pan"/>
-      <origin xyz="0 0 ${joint_pan_z}" rpy="0.0 0.0 0.0"/>
+      <origin xyz="0 0 ${joint_pan_pos_z}" rpy="0.0 0.0 0.0"/>
       <limit effort="0" lower="${pan_lower}" upper="${pan_upper}" velocity="0"/>
       <axis xyz="0 0 1"/>
+      <dynamics damping="${ptu_damping}" friction="${ptu_friction}"/>
     </joint>
     <!-- PAN LINK -->
@@ -86,21 +100,35 @@
         </geometry>
       </visual>
+      <!-- TILT MOTOR -->
+      <visual>
+        <origin xyz="0.0 0.03 ${joint_tilt_pos_z}" rpy="${pi/2} 0 0"/>
+        <geometry>
+          <cylinder length="0.06" radius="0.011"/>
+        </geometry>
+      </visual>
+      <collision>
+        <origin xyz="0.0 0.03 ${joint_tilt_pos_z}" rpy="${pi/2} 0 0"/>
+        <geometry>
+          <cylinder length="0.06" radius="0.011"/>
+        </geometry>
+      </collision>
     </link>
     <!-- TILT JOINT -->
-    <joint name="tilt" type="revolute">
-      <parent link="mast"/>
-      <child link="link_pan"/>
-      <origin xyz="0 0 ${mast_l}" rpy="0.0 0.0 0.0"/>
+    <joint name="joint_STR_tilt" type="revolute">
+      <parent link="link_pan"/>
+      <child link="link_tilt"/>
+      <origin xyz="0 0 ${joint_tilt_pos_z}" rpy="${joint_tilt_rot_x} 0.0 0.0"/>
       <limit effort="0" lower="${tilt_lower}" upper="${tilt_upper}" velocity="0"/>
       <axis xyz="0 0 1"/>
+      <dynamics damping="${ptu_damping}" friction="${ptu_friction}"/>
     </joint>
-<!--
-    <link name="link_bogie_${position}">
+    <!-- TILT LINK -->
+    <link name="link_tilt">
       <inertial>
-        <mass value="${bogie_mass}"/>
-        <inertia
-              ixx="${bogie_mass / 12.0 * (3 * bogie_r * bogie_r + bogie_l * bogie_l)}"
-              iyy="${bogie_mass / 12.0 * (3 * bogie_r * bogie_r + bogie_l * bogie_l)}"
-              izz="${bogie_mass /  2.0 *  bogie_r * bogie_r}"
+        <mass value="${link_tilt_mass}"/>
+          <inertia
+              ixx="${link_tilt_mass / 12.0 * (link_tilt_y * link_tilt_z / 2)}"
+              iyy="${link_tilt_mass / 12.0 * (link_tilt_x * link_tilt_z / 2)}"
+              izz="${link_tilt_mass / 12.0 * (link_tilt_x * link_tilt_y / 2)}"
               ixy="0"
               ixz="0"
@@ -108,17 +136,16 @@
       </inertial>
       <collision>
-        <origin xyz="0 0 0" rpy="0 ${pi / 2} 0"/>
+        <origin xyz="${link_tilt_pos_x} ${link_tilt_pos_y} ${link_tilt_pos_z}" rpy="0 0 0"/>
         <geometry>
-          <xacro:insert_block name="geometry" />
+          <box size="${link_tilt_x} ${link_tilt_y} ${link_tilt_z}"/>
         </geometry>
       </collision>
       <visual>
-        <origin xyz="0 0 0" rpy="0 ${pi / 2} 0"/>
+        <origin xyz="${link_tilt_pos_x} ${link_tilt_pos_y} ${link_tilt_pos_z}" rpy="0 0 0"/>
         <geometry>
-          <xacro:insert_block name="geometry" />
+          <box size="${link_tilt_x} ${link_tilt_y} ${link_tilt_z}"/>
         </geometry>
       </visual>
     </link>
- -->
   </xacro:macro>
 </robot>

Commit message: added camera, but it is not stable or polished

File: urdf/ptu.xacro (robot description, xacro)
@@ -28,6 +28,6 @@
     <xacro:property name="joint_tilt_pos_z" value="0.0265" />
     <xacro:property name="joint_tilt_rot_x" value="${pi/2}" />
-    <!-- PAN LINK -->
-    <xacro:property name="link_tilt_mass" value="0.1" />
+    <!-- TILT LINK -->
+    <xacro:property name="link_tilt_mass" value="1.0" />
     <xacro:property name="link_tilt_x" value="0.022" />
     <xacro:property name="link_tilt_y" value="0.0035" />
@@ -36,4 +36,15 @@
     <xacro:property name="link_tilt_pos_y" value="0.01625" />
     <xacro:property name="link_tilt_pos_z" value="0.0" />
+    <!-- CAM JOINT -->
+    <xacro:property name="joint_cam_pos_y" value="0.036" />
+    <xacro:property name="joint_cam_rot_x" value="${pi/2}" />
+    <!-- CAM LINK -->
+    <xacro:property name="link_cam_mass" value="1.0" />
+    <xacro:property name="link_cam_x" value="0.022" />
+    <xacro:property name="link_cam_y" value="0.0035" />
+    <xacro:property name="link_cam_z" value="0.072" />
+    <xacro:property name="link_cam_pos_x" value="0.0" />
+    <xacro:property name="link_cam_pos_y" value="0.01625" />
+    <xacro:property name="link_cam_pos_z" value="0.0" />
     <!-- MAST JOINT -->
     <joint name="ptu_base" type="fixed">
@@ -148,4 +159,68 @@
       </visual>
     </link>
+    <!-- CAMERA -->
+    <joint name="camera_joint" type="fixed">
+        <parent link="link_tilt"/>
+        <child link="link_cam"/>
+        <origin rpy="0 0 0" xyz="0.0 ${joint_cam_pos_y} 0.0"/>
+        <axis xyz="1 0 0" />
+    </joint>
+    <!-- CAMERA LINK -->
+    <link name="link_cam">
+      <inertial>
+        <mass value="${link_cam_mass}"/>
+          <inertia
+              ixx="${link_cam_mass / 12.0 * (link_cam_y * link_cam_z / 2)}"
+              iyy="${link_cam_mass / 12.0 * (link_cam_x * link_cam_z / 2)}"
+              izz="${link_cam_mass / 12.0 * (link_cam_x * link_cam_y / 2)}"
+              ixy="0"
+              ixz="0"
+              iyz="0"/>
+      </inertial>
+      <collision>
+        <origin xyz="${link_cam_pos_x} ${link_cam_pos_y} ${link_cam_pos_z}" rpy="0 0 0"/>
+        <geometry>
+          <box size="${link_cam_x} ${link_cam_y} ${link_cam_z}"/>
+        </geometry>
+      </collision>
+      <visual>
+        <origin xyz="${link_cam_pos_x} ${link_cam_pos_y} ${link_cam_pos_z}" rpy="0 0 0"/>
+        <geometry>
+          <box size="${link_cam_x} ${link_cam_y} ${link_cam_z}"/>
+        </geometry>
+      </visual>
+    </link>
+    <gazebo reference="link_cam">
+      <sensor type="camera" name="camera_camera_sensor">
+        <update_rate>30.0</update_rate>
+        <camera>
+          <pose>0.035 0 0.078 0 ${-pi/2} 0</pose>
+          <horizontal_fov>${85 * pi/180.0}</horizontal_fov>
+          <image>
+            <format>R8G8B8</format>
+            <width>1020</width>
+            <height>1020</height>
+          </image>
+          <clip>
+            <near>0.01</near>
+            <far>100</far>
+          </clip>
+        </camera>
+        <plugin name="camera_camera_controller" filename="libgazebo_ros_camera.so">
+          <alwaysOn>true</alwaysOn>
+          <updateRate>0.0</updateRate>
+          <cameraName>camera</cameraName>
+          <imageTopicName>image_raw</imageTopicName>
+          <cameraInfoTopicName>camera_info</cameraInfoTopicName>
+          <frameName>camera_link</frameName>
+          <hackBaseline>0.07</hackBaseline>
+          <distortionK1>0.0</distortionK1>
+          <distortionK2>0.0</distortionK2>
+          <distortionK3>0.0</distortionK3>
+          <distortionT1>0.0</distortionT1>
+          <distortionT2>0.0</distortionT2>
+        </plugin>
+      </sensor>
+    </gazebo>
   </xacro:macro>
 </robot>

Commit message: fixed pan and tilt joint until gazebo plugin is updated. Add link for BB2 and moved camera to gazebo file

File: urdf/ptu.xacro (robot description, xacro)
@@ -5,5 +5,4 @@
     <xacro:property name="ptu_damping" value="2" />
     <xacro:property name="ptu_friction" value="0.1" />
-    <xacro:include filename="$(find rover_config)/urdf/ptu.gazebo" />
     <!-- PARAMETERS -->
     <!-- MAST LINK -->
@@ -41,7 +40,8 @@
     <!-- CAM LINK -->
     <xacro:property name="link_cam_mass" value="1.0" />
-    <xacro:property name="link_cam_x" value="0.022" />
-    <xacro:property name="link_cam_y" value="0.0035" />
-    <xacro:property name="link_cam_z" value="0.072" />
+    <xacro:property name="link_cam_x" value="0.0474" />
+    <xacro:property name="link_cam_y" value="0.157" />
+    <xacro:property name="link_cam_z" value="0.036" />
+    <xacro:property name="link_cam_rot_r" value="${-pi/2}" />
     <xacro:property name="link_cam_pos_x" value="0.0" />
     <xacro:property name="link_cam_pos_y" value="0.01625" />
@@ -79,5 +79,5 @@
     </link>
     <!-- PAN JOINT -->
-    <joint name="joint_STR_pan" type="revolute">
+    <joint name="joint_PAN" type="fixed">
       <parent link="link_mast"/>
       <child link="link_pan"/>
@@ -126,5 +126,5 @@
     </link>
     <!-- TILT JOINT -->
-    <joint name="joint_STR_tilt" type="revolute">
+    <joint name="joint_TLT" type="fixed">
       <parent link="link_pan"/>
       <child link="link_tilt"/>
@@ -163,5 +163,5 @@
         <parent link="link_tilt"/>
         <child link="link_cam"/>
-        <origin rpy="0 0 0" xyz="0.0 ${joint_cam_pos_y} 0.0"/>
+        <origin rpy="${link_cam_rot_r} 0 0" xyz="0.0 ${joint_cam_pos_y} 0.0"/>
         <axis xyz="1 0 0" />
     </joint>
@@ -191,36 +191,5 @@
       </visual>
     </link>
-    <gazebo reference="link_cam">
-      <sensor type="camera" name="camera_camera_sensor">
-        <update_rate>30.0</update_rate>
-        <camera>
-          <pose>0.035 0 0.078 0 ${-pi/2} 0</pose>
-          <horizontal_fov>${85 * pi/180.0}</horizontal_fov>
-          <image>
-            <format>R8G8B8</format>
-            <width>1020</width>
-            <height>1020</height>
-          </image>
-          <clip>
-            <near>0.01</near>
-            <far>100</far>
-          </clip>
-        </camera>
-        <plugin name="camera_camera_controller" filename="libgazebo_ros_camera.so">
-          <alwaysOn>true</alwaysOn>
-          <updateRate>0.0</updateRate>
-          <cameraName>camera</cameraName>
-          <imageTopicName>image_raw</imageTopicName>
-          <cameraInfoTopicName>camera_info</cameraInfoTopicName>
-          <frameName>camera_link</frameName>
-          <hackBaseline>0.07</hackBaseline>
-          <distortionK1>0.0</distortionK1>
-          <distortionK2>0.0</distortionK2>
-          <distortionK3>0.0</distortionK3>
-          <distortionT1>0.0</distortionT1>
-          <distortionT2>0.0</distortionT2>
-        </plugin>
-      </sensor>
-    </gazebo>
+    <xacro:include filename="$(find rover_config)/urdf/ptu.gazebo" />
   </xacro:macro>
 </robot>

Commit message: added generic bb2 camera model, added bb2 as nav_cam

File: urdf/ptu.xacro (robot description, xacro)
@@ -2,4 +2,5 @@
 <robot xmlns:xacro="http://wiki.ros.org/xacro">
   <xacro:macro name="ptu" params="parent_link *origin">
+    <xacro:include filename="$(find rover_config)/urdf/ptu.gazebo" />
     <!-- PHYSICS -->
     <xacro:property name="ptu_damping" value="2" />
@@ -37,14 +38,5 @@
     <!-- CAM JOINT -->
     <xacro:property name="joint_cam_pos_y" value="0.036" />
-    <xacro:property name="joint_cam_rot_x" value="${pi/2}" />
-    <!-- CAM LINK -->
-    <xacro:property name="link_cam_mass" value="1.0" />
-    <xacro:property name="link_cam_x" value="0.0474" />
-    <xacro:property name="link_cam_y" value="0.157" />
-    <xacro:property name="link_cam_z" value="0.036" />
-    <xacro:property name="link_cam_rot_r" value="${-pi/2}" />
-    <xacro:property name="link_cam_pos_x" value="0.0" />
-    <xacro:property name="link_cam_pos_y" value="0.01625" />
-    <xacro:property name="link_cam_pos_z" value="0.0" />
+    <xacro:property name="joint_cam_rot_r" value="${-pi/2}" />
     <!-- MAST JOINT -->
     <joint name="ptu_base" type="fixed">
@@ -159,37 +151,8 @@
       </visual>
     </link>
-    <!-- CAMERA -->
-    <joint name="camera_joint" type="fixed">
-        <parent link="link_tilt"/>
-        <child link="link_cam"/>
-        <origin rpy="${link_cam_rot_r} 0 0" xyz="0.0 ${joint_cam_pos_y} 0.0"/>
-        <axis xyz="1 0 0" />
-    </joint>
-    <!-- CAMERA LINK -->
-    <link name="link_cam">
-      <inertial>
-        <mass value="${link_cam_mass}"/>
-          <inertia
-              ixx="${link_cam_mass / 12.0 * (link_cam_y * link_cam_z / 2)}"
-              iyy="${link_cam_mass / 12.0 * (link_cam_x * link_cam_z / 2)}"
-              izz="${link_cam_mass / 12.0 * (link_cam_x * link_cam_y / 2)}"
-              ixy="0"
-              ixz="0"
-              iyz="0"/>
-      </inertial>
-      <collision>
-        <origin xyz="${link_cam_pos_x} ${link_cam_pos_y} ${link_cam_pos_z}" rpy="0 0 0"/>
-        <geometry>
-          <box size="${link_cam_x} ${link_cam_y} ${link_cam_z}"/>
-        </geometry>
-      </collision>
-      <visual>
-        <origin xyz="${link_cam_pos_x} ${link_cam_pos_y} ${link_cam_pos_z}" rpy="0 0 0"/>
-        <geometry>
-          <box size="${link_cam_x} ${link_cam_y} ${link_cam_z}"/>
-        </geometry>
-      </visual>
-    </link>
-    <xacro:include filename="$(find rover_config)/urdf/ptu.gazebo" />
+    <xacro:include filename="$(find rover_config)/urdf/bb2.xacro" />
+    <xacro:bb2 name="nav_cam" parent_link="link_tilt">
+        <origin rpy="${joint_cam_rot_r} 0 0" xyz="0.0 ${joint_cam_pos_y} 0.0"/>
+    </xacro:bb2>
   </xacro:macro>
 </robot>

Commit message: Make PTU tilt coordinate system follow convention

File: urdf/ptu.xacro (robot description, xacro)
@@ -31,5 +31,5 @@
     <xacro:property name="joint_tilt_pos_y" value="-0.0095" />
     <xacro:property name="joint_tilt_pos_z" value="0.0295" />
-    <xacro:property name="joint_tilt_rot_x" value="${pi/2}" />
+    <xacro:property name="joint_tilt_rot_x" value="${-pi/2}" />
     <!-- TILT LINK -->
     <xacro:property name="link_tilt_mass" value="0.1" />
@@ -38,10 +38,10 @@
     <xacro:property name="link_tilt_z" value="0.072" />
     <xacro:property name="link_tilt_pos_x" value="0.0" />
-    <xacro:property name="link_tilt_pos_y" value="${0.01625 - link_tilt_y}" />
-    <xacro:property name="link_tilt_pos_z" value="${joint_tilt_pos_y}" />
+    <xacro:property name="link_tilt_pos_y" value="${- 0.01625 + link_tilt_y}" />
+    <xacro:property name="link_tilt_pos_z" value="${-joint_tilt_pos_y}" />
     <!-- CAM JOINT -->
-    <xacro:property name="joint_cam_pos_y" value="0.015" />
-    <xacro:property name="joint_cam_pos_z" value="${joint_tilt_pos_y}" />
-    <xacro:property name="joint_cam_rot_r" value="${-pi/2}" />
+    <xacro:property name="joint_cam_pos_y" value="-0.015" />
+    <xacro:property name="joint_cam_pos_z" value="${-joint_tilt_pos_y}" />
+    <xacro:property name="joint_cam_rot_r" value="${pi/2}" />
     <!-- MAST JOINT -->
     <joint name="ptu_base" type="fixed">
