Commit message: added deployment joint to URDF

File: urdf/marta.xacro (robot description, xacro)
@@ -1,4 +1,4 @@
 <?xml version="1.0"?>
-<robot name="rover_dummy" xmlns:xacro="http://www.ros.org/wiki/xacro">
+<robot name="marta" xmlns:xacro="http://www.ros.org/wiki/xacro">
   <xacro:property name="mass" value="1.0" />
   <xacro:property name="damping" value="0.1" />
@@ -42,14 +42,14 @@
   </link>
   <!-- Definition for a wheel assembly -->
-  <xacro:macro name="wheel_assembly" params="position *origin_DEP">
-    <joint name="joint_DEP_${position}" type="fixed">
+  <xacro:macro name="wheel_assembly" params="position configuration *origin">
+    <joint name="joint_deploy_${position}" type="revolute">
       <parent link="base_link"/>
-      <child link="link_DEP_${position}"/>
+      <child link="link_${position}"/>
       <limit effort="${limit_steer_effort}" lower="${limit_steer_lower}" upper="${limit_steer_upper}" velocity="${limit_steer_velocity}"/>
-      <xacro:insert_block name="origin_DEP" />
-      <axis xyz="0 1 0"/>
+      <xacro:insert_block name="origin" />
+      <axis xyz="0 0 1"/>
       <dynamics damping="${damping}" friction="${friction}"/>
     </joint>
-    <link name="link_DEP_${position}">
+    <link name="link_deploy_${position}">
       <collision>
         <origin xyz="0 0 0" rpy="0 0 0"/>
@@ -75,13 +75,13 @@
       </visual>
     </link>
-    <joint name="joint_STR_${position}" type="fixed">
-      <parent link="link_DEP_${position}"/>
-      <child link="link_STR_${position}"/>
+    <joint name="joint_steer_${position}" type="revolute">
+      <parent link="base_link"/>
+      <child link="link_${position}"/>
       <limit effort="${limit_steer_effort}" lower="${limit_steer_lower}" upper="${limit_steer_upper}" velocity="${limit_steer_velocity}"/>
-      <origin xyz="-0.15 0 0.15" rpy="-1.57 0 0"/>
+      <xacro:insert_block name="origin" />
       <axis xyz="0 0 1"/>
       <dynamics damping="${damping}" friction="${friction}"/>
     </joint>
-    <link name="link_STR_${position}">
+    <link name="link_steer_${position}">
       <collision>
         <origin xyz="0 0 0" rpy="0 0 0"/>
@@ -107,13 +107,13 @@
       </visual>
     </link>
-    <joint name="joint_DRV_${position}" type="fixed">
-      <parent link="link_STR_${position}"/>
-      <child link="link_DRV_${position}"/>
+    <joint name="joint_drive_${position}" type="continuous">
+      <parent link="link_${position}"/>
+      <child link="wheel_${position}"/>
       <limit effort="${limit_drive_effort}" velocity="${limit_drive_velocity}"/>
-      <origin xyz="0 0 ${-size_link / 2 - 2 * wheel_radius}" rpy="-1.57 0 0"/>
+      <origin xyz="0 0 ${-size_link / 2 - 2 * wheel_radius}" rpy="0 0 0"/>
       <axis xyz="0 1 0"/>
       <dynamics damping="${damping}" friction="${friction}"/>
     </joint>
-    <link name="link_DRV_${position}">
+    <link name="wheel_${position}">
       <collision>
         <origin xyz="0 0 0" rpy="${pi / 2} 0 0"/>
@@ -139,19 +139,19 @@
       </visual>
     </link>
-    <transmission name=" _STR_${position}">
+    <transmission name=" _steer_${position}">
       <type>transmission_interface/SimpleTransmission</type>
-      <joint name="joint_STR_${position}">
+      <joint name="joint_steer_${position}">
         <hardwareInterface>hardware_interface/EffortJointInterface</hardwareInterface>
       </joint>
-      <actuator name="motor_STR_${position}">
+      <actuator name="motor_steer_${position}">
         <mechanicalReduction>1</mechanicalReduction>
       </actuator>
     </transmission>
-    <transmission name="transmission_DRV_${position}">
+    <transmission name="transmission_drive_${position}">
       <type>transmission_interface/SimpleTransmission</type>
-      <joint name="joint_DRV_${position}">
+      <joint name="joint_drive_${position}">
         <hardwareInterface>hardware_interface/EffortJointInterface</hardwareInterface>
       </joint>
-      <actuator name="motor_DRV_${position}">
+      <actuator name="motor_drive_${position}">
         <mechanicalReduction>1</mechanicalReduction>
       </actuator>
@@ -159,22 +159,21 @@
   </xacro:macro>
   <!-- Define all the wheel assemblies as set their positions -->
-  <xacro:wheel_assembly position="RF">
+  <xacro:wheel_assembly position="back_left">
+    <origin xyz="${-(size_base / 2 + size_link)} ${(size_base / 2 + size_link)} 0" rpy="0 0 0"/>
+  </xacro:wheel_assembly>
+  <xacro:wheel_assembly position="back_right">
+    <origin xyz="${-(size_base / 2 + size_link)} ${-(size_base / 2 + size_link)} 0" rpy="0 0 0"/>
+  </xacro:wheel_assembly>
+  <xacro:wheel_assembly position="center_left">
+    <origin xyz="0 ${(size_base / 2 + size_link)} 0" rpy="0 0 0"/>
+  </xacro:wheel_assembly>
+  <xacro:wheel_assembly position="center_right">
+    <origin xyz="0 ${-(size_base / 2 + size_link)} 0" rpy="0 0 0"/>
+  </xacro:wheel_assembly>
+  <xacro:wheel_assembly position="front_left">
+    <origin xyz="${(size_base / 2 + size_link)} ${(size_base / 2 + size_link)} 0" rpy="0 0 0"/>
+  </xacro:wheel_assembly>
+  <xacro:wheel_assembly position="front_right">
     <origin xyz="${(size_base / 2 + size_link)} ${-(size_base / 2 + size_link)} 0" rpy="0 0 0"/>
   </xacro:wheel_assembly>
-  <xacro:wheel_assembly position="RM">
-    <origin xyz="0 ${-(size_base / 2 + size_link)} 0" rpy="0 0 0"/>
-  </xacro:wheel_assembly>
-  <xacro:wheel_assembly position="RR">
-    <!-- <origin xyz="${-(size_base / 2 + size_link)} ${-(size_base / 2 + size_link)} 0" rpy="0 0 0"/> -->
-    <origin xyz="${-(size_base / 2 + size_link)} ${-(size_base / 2 + size_link)} 0" rpy="1.57 0 0"/>
-  </xacro:wheel_assembly>
-  <xacro:wheel_assembly position="LF">
-    <origin xyz="${(size_base / 2 + size_link)} ${(size_base / 2 + size_link)} 0" rpy="0 0 0"/>
-  </xacro:wheel_assembly>
-  <xacro:wheel_assembly position="LM">
-    <origin xyz="0 ${(size_base / 2 + size_link)} 0" rpy="0 0 0"/>
-  </xacro:wheel_assembly>
-  <xacro:wheel_assembly position="LR">
-    <origin xyz="${-(size_base / 2 + size_link)} ${(size_base / 2 + size_link)} 0" rpy="1.57 0 0"/>
-  </xacro:wheel_assembly>
 </robot>

Commit message: added a marta representative locomotion system.

File: urdf/marta.xacro (robot description, xacro)
@@ -1,11 +1,12 @@
 <?xml version="1.0"?>
-<robot name="marta" xmlns:xacro="http://www.ros.org/wiki/xacro">
+<robot name="rover_dummy" xmlns:xacro="http://www.ros.org/wiki/xacro">
   <xacro:property name="mass" value="1.0" />
   <xacro:property name="damping" value="0.1" />
   <xacro:property name="friction" value="0.1" />
-  <xacro:property name="size_base" value="1.0" />
-  <xacro:property name="size_link" value="0.25" />
+  <xacro:property name="size_base" value="0.5" />
+  <xacro:property name="size_link" value="0.15" />
   <!-- Warning: the wheel_radius value must be the same as in the YAML configuration file-->
-  <xacro:property name="wheel_radius" value="${size_link / 2}" />
+  <xacro:property name="wheel_radius" value="0.08" />
+  <xacro:property name="variant" value="1.0" />
   <xacro:property name="limit_drive_effort" value="100.0" />
   <xacro:property name="limit_drive_velocity" value="1.0" />
@@ -14,4 +15,6 @@
   <xacro:property name="limit_steer_upper" value="${pi / 2}" />
   <xacro:property name="limit_steer_velocity" value="1.0" />
+  <xacro:property name="side_boogie_lower" value="${-pi / 2}" />
+  <xacro:property name="side_boogie_upper" value="${pi / 2}" />
   <!-- Import all Gazebo-customization elements, including Gazebo colors and plugins -->
   <xacro:include filename="$(find rover_config)/urdf/rover_dummy.gazebo" />
@@ -19,5 +22,5 @@
   <link name="base_link">
     <collision>
-      <origin xyz="0 0 0" rpy="0 0 0"/>
+      <origin xyz="0 0 ${size_base / 4}" rpy="0 0 0"/>
       <geometry>
         <box size="${size_base} ${size_base} ${size_base / 2}"/>
@@ -35,5 +38,5 @@
     </inertial>
     <visual>
-      <origin xyz="0 0 0" rpy="0 0 0"/>
+      <origin xyz="0 0 ${size_base / 4}" rpy="0 0 0"/>
       <geometry>
         <box size="${size_base} ${size_base} ${size_base / 2}"/>
@@ -41,15 +44,50 @@
     </visual>
   </link>
+  <!-- Definition for a side boogie assembly -->
+  <xacro:macro name="boogie" params="position *origin_boogie">
+    <xacro:property name="boogie_link" value="link_boogie_${position}" />
+    <joint name="joint_boogie_${position}" type="fixed">
+      <parent link="base_link"/>
+      <child link="link_boogie_${position}"/>
+      <xacro:insert_block name="origin_boogie" />
+      <limit effort="0" lower="${side_boogie_lower}" upper="${side_boogie_upper}" velocity="0"/>
+      <axis xyz="0 0 1"/>
+    </joint>
+    <link name="link_boogie_${position}">
+      <collision>
+        <origin xyz="0 0 0.03" rpy="0 ${pi / 2} 0"/>
+        <geometry>
+          <cylinder length="0.5" radius="0.04"/>
+        </geometry>
+      </collision>
+      <inertial>
+        <mass value="${mass}"/>
+        <inertia
+              ixx="${mass / 12.0 * (size_link * size_link / 2)}"
+              iyy="${mass / 12.0 * (size_link * size_link / 2)}"
+              izz="${mass / 12.0 * (size_link * size_link / 2)}"
+              ixy="0"
+              ixz="0"
+              iyz="0"/>
+      </inertial>
+      <visual>
+        <origin xyz="0 0 0.03" rpy="0 ${pi / 2} 0"/>
+        <geometry>
+          <cylinder length="0.5" radius="0.04"/>
+        </geometry>
+      </visual>
+    </link>
+  </xacro:macro>
   <!-- Definition for a wheel assembly -->
-  <xacro:macro name="wheel_assembly" params="position configuration *origin">
-    <joint name="joint_deploy_${position}" type="revolute">
-      <parent link="base_link"/>
-      <child link="link_${position}"/>
+  <xacro:macro name="wheel_assembly" params="position boogie_name *origin_DEP *origin_STR">
+    <joint name="joint_DEP_${position}" type="fixed">
+      <parent link="link_boogie_${boogie_name}"/>
+      <child link="link_DEP_${position}"/>
       <limit effort="${limit_steer_effort}" lower="${limit_steer_lower}" upper="${limit_steer_upper}" velocity="${limit_steer_velocity}"/>
-      <xacro:insert_block name="origin" />
+      <xacro:insert_block name="origin_DEP" />
       <axis xyz="0 0 1"/>
       <dynamics damping="${damping}" friction="${friction}"/>
     </joint>
-    <link name="link_deploy_${position}">
+    <link name="link_DEP_${position}">
       <collision>
         <origin xyz="0 0 0" rpy="0 0 0"/>
@@ -75,13 +113,14 @@
       </visual>
     </link>
-    <joint name="joint_steer_${position}" type="revolute">
-      <parent link="base_link"/>
-      <child link="link_${position}"/>
+    <joint name="joint_STR_${position}" type="fixed">
+      <parent link="link_DEP_${position}"/>
+      <child link="link_STR_${position}"/>
       <limit effort="${limit_steer_effort}" lower="${limit_steer_lower}" upper="${limit_steer_upper}" velocity="${limit_steer_velocity}"/>
-      <xacro:insert_block name="origin" />
+      <!-- <origin xyz="0.15 0 0.15" rpy="${pi / 2} 0 0"/> -->
+      <xacro:insert_block name="origin_STR" />
       <axis xyz="0 0 1"/>
       <dynamics damping="${damping}" friction="${friction}"/>
     </joint>
-    <link name="link_steer_${position}">
+    <link name="link_STR_${position}">
       <collision>
         <origin xyz="0 0 0" rpy="0 0 0"/>
@@ -107,15 +146,15 @@
       </visual>
     </link>
-    <joint name="joint_drive_${position}" type="continuous">
-      <parent link="link_${position}"/>
-      <child link="wheel_${position}"/>
+    <joint name="joint_DRV_${position}" type="fixed">
+      <parent link="link_STR_${position}"/>
+      <child link="link_DRV_${position}"/>
       <limit effort="${limit_drive_effort}" velocity="${limit_drive_velocity}"/>
-      <origin xyz="0 0 ${-size_link / 2 - 2 * wheel_radius}" rpy="0 0 0"/>
-      <axis xyz="0 1 0"/>
+      <origin xyz="0 0 ${-size_link / 2 - 1.1 * wheel_radius}" rpy="-1.57 0 0"/>
+      <axis xyz="0 0 1"/>
       <dynamics damping="${damping}" friction="${friction}"/>
     </joint>
-    <link name="wheel_${position}">
-      <collision>
-        <origin xyz="0 0 0" rpy="${pi / 2} 0 0"/>
+    <link name="link_DRV_${position}">
+      <collision>
+        <origin xyz="0 0 0" rpy="0 0 0"/>
         <geometry>
           <cylinder length="${size_link}" radius="${wheel_radius}"/>
@@ -133,5 +172,5 @@
       </inertial>
       <visual>
-        <origin xyz="0 0 0" rpy="${pi / 2} 0 0"/>
+        <origin xyz="0 0 0" rpy="0 0 0"/>
         <geometry>
           <cylinder length="${size_link}" radius="${wheel_radius}"/>
@@ -139,19 +178,19 @@
       </visual>
     </link>
-    <transmission name=" _steer_${position}">
+    <transmission name="_STR_${position}">
       <type>transmission_interface/SimpleTransmission</type>
-      <joint name="joint_steer_${position}">
+      <joint name="joint_STR_${position}">
         <hardwareInterface>hardware_interface/EffortJointInterface</hardwareInterface>
       </joint>
-      <actuator name="motor_steer_${position}">
+      <actuator name="motor_STR_${position}">
         <mechanicalReduction>1</mechanicalReduction>
       </actuator>
     </transmission>
-    <transmission name="transmission_drive_${position}">
+    <transmission name="transmission_DRV_${position}">
       <type>transmission_interface/SimpleTransmission</type>
-      <joint name="joint_drive_${position}">
+      <joint name="joint_DRV_${position}">
         <hardwareInterface>hardware_interface/EffortJointInterface</hardwareInterface>
       </joint>
-      <actuator name="motor_drive_${position}">
+      <actuator name="motor_DRV_${position}">
         <mechanicalReduction>1</mechanicalReduction>
       </actuator>
@@ -159,21 +198,42 @@
   </xacro:macro>
   <!-- Define all the wheel assemblies as set their positions -->
-  <xacro:wheel_assembly position="back_left">
-    <origin xyz="${-(size_base / 2 + size_link)} ${(size_base / 2 + size_link)} 0" rpy="0 0 0"/>
-  </xacro:wheel_assembly>
-  <xacro:wheel_assembly position="back_right">
-    <origin xyz="${-(size_base / 2 + size_link)} ${-(size_base / 2 + size_link)} 0" rpy="0 0 0"/>
-  </xacro:wheel_assembly>
-  <xacro:wheel_assembly position="center_left">
-    <origin xyz="0 ${(size_base / 2 + size_link)} 0" rpy="0 0 0"/>
-  </xacro:wheel_assembly>
-  <xacro:wheel_assembly position="center_right">
-    <origin xyz="0 ${-(size_base / 2 + size_link)} 0" rpy="0 0 0"/>
-  </xacro:wheel_assembly>
-  <xacro:wheel_assembly position="front_left">
-    <origin xyz="${(size_base / 2 + size_link)} ${(size_base / 2 + size_link)} 0" rpy="0 0 0"/>
-  </xacro:wheel_assembly>
-  <xacro:wheel_assembly position="front_right">
-    <origin xyz="${(size_base / 2 + size_link)} ${-(size_base / 2 + size_link)} 0" rpy="0 0 0"/>
+  <!-- LEFT BOGIE  -->
+  <xacro:property name="side_boogie_left_name" value="LFB" />
+  <xacro:boogie position="${side_boogie_left_name}">
+    <origin xyz="0.3 ${size_base / 2} 0" rpy="${- pi / 2} 0 0"/>
+  </xacro:boogie>
+  <xacro:wheel_assembly position="LF" boogie_name="${side_boogie_left_name}">
+    <origin xyz="0.2 0 0.05" rpy="0 0 0"/>
+    <origin xyz="0.1 0 0.1" rpy="${pi / 2} 0 0"/>
+  </xacro:wheel_assembly>
+  <xacro:wheel_assembly position="LM" boogie_name="${side_boogie_left_name}">
+    <origin xyz="-0.2 0 0.05" rpy="0 0 0"/>
+    <origin xyz="-0.1 0 0.1" rpy="${pi / 2} 0 0"/>
+  </xacro:wheel_assembly>
+  <!-- RIGHT BOGIE  -->
+  <xacro:property name="side_boogie_right_name" value="RFB" />
+  <xacro:boogie position="${side_boogie_right_name}">
+    <origin xyz="0.3 -${size_base / 2} 0" rpy="${- pi / 2} 0 ${pi}"/>
+  </xacro:boogie>
+  <xacro:wheel_assembly position="RF" boogie_name="${side_boogie_right_name}">
+    <origin xyz="-0.2 0 0.05" rpy="0 0 0"/>
+    <origin xyz="-0.1 0 0.1" rpy="${pi / 2} 0 0"/>
+  </xacro:wheel_assembly>
+  <xacro:wheel_assembly position="RM" boogie_name="${side_boogie_right_name}">
+    <origin xyz="0.2 0 0.05" rpy="0 0 0"/>
+    <origin xyz="0.1 0 0.1" rpy="${pi / 2} 0 0"/>
+  </xacro:wheel_assembly>
+  <!-- REAR BOGIE  -->
+  <xacro:property name="side_boogie_rear_name" value="MRB" />
+  <xacro:boogie position="${side_boogie_rear_name}">
+    <origin xyz="-${size_base / 2 + 0.05} 0 0" rpy="${- pi / 2} 0 ${pi / 2}"/>
+  </xacro:boogie>
+  <xacro:wheel_assembly position="RR" boogie_name="${side_boogie_rear_name}">
+    <origin xyz="-0.3 0 0.05" rpy="0 ${3 * pi / 2} 0"/>
+    <origin xyz="0.1 0 0.1" rpy="${pi / 2} 0 0"/>
+  </xacro:wheel_assembly>
+  <xacro:wheel_assembly position="LR" boogie_name="${side_boogie_rear_name}">
+    <origin xyz="0.3 0 0.05" rpy="0 ${pi / 2} 0"/>
+    <origin xyz="-0.1 0 0.1" rpy="${pi / 2} 0 0"/>
   </xacro:wheel_assembly>
 </robot>

Commit message: changed joints from fixed to revolute and continuous

File: urdf/marta.xacro (robot description, xacro)
@@ -15,6 +15,6 @@
   <xacro:property name="limit_steer_upper" value="${pi / 2}" />
   <xacro:property name="limit_steer_velocity" value="1.0" />
-  <xacro:property name="side_boogie_lower" value="${-pi / 2}" />
-  <xacro:property name="side_boogie_upper" value="${pi / 2}" />
+  <xacro:property name="side_boogie_lower" value="${-pi / 4}" />
+  <xacro:property name="side_boogie_upper" value="${pi / 4}" />
   <!-- Import all Gazebo-customization elements, including Gazebo colors and plugins -->
   <xacro:include filename="$(find rover_config)/urdf/marta.gazebo" />
@@ -47,5 +47,5 @@
   <xacro:macro name="boogie" params="position *origin_boogie">
     <xacro:property name="boogie_link" value="link_boogie_${position}" />
-    <joint name="joint_boogie_${position}" type="fixed">
+    <joint name="joint_boogie_${position}" type="revolute">
       <parent link="base_link"/>
       <child link="link_boogie_${position}"/>
@@ -81,5 +81,5 @@
   <!-- Definition for a wheel assembly -->
   <xacro:macro name="wheel_assembly" params="position boogie_name *origin_DEP *origin_STR">
-    <joint name="joint_DEP_${position}" type="fixed">
+    <joint name="joint_DEP_${position}" type="revolute">
       <parent link="link_boogie_${boogie_name}"/>
       <child link="link_DEP_${position}"/>
@@ -113,5 +113,5 @@
       </visual>
     </link>
-    <joint name="joint_STR_${position}" type="fixed">
+    <joint name="joint_STR_${position}" type="revolute">
       <parent link="link_DEP_${position}"/>
       <child link="link_STR_${position}"/>
@@ -146,5 +146,5 @@
       </visual>
     </link>
-    <joint name="joint_DRV_${position}" type="fixed">
+    <joint name="joint_DRV_${position}" type="continuous">
       <parent link="link_STR_${position}"/>
       <child link="link_DRV_${position}"/>

Commit message: added driving direction to flip direction of deployment and driving joint

File: urdf/marta.xacro (robot description, xacro)
@@ -80,5 +80,6 @@
   </xacro:macro>
   <!-- Definition for a wheel assembly -->
-  <xacro:macro name="wheel_assembly" params="position boogie_name *origin_DEP *origin_STR">
+  <!-- Driving direction is used to invert the direction of the deployment and driving joint -->
+  <xacro:macro name="wheel_assembly" params="position boogie_name driving_direction *origin_DEP *origin_STR">
     <joint name="joint_DEP_${position}" type="revolute">
       <parent link="link_boogie_${boogie_name}"/>
@@ -86,5 +87,5 @@
       <limit effort="${limit_steer_effort}" lower="${limit_steer_lower}" upper="${limit_steer_upper}" velocity="${limit_steer_velocity}"/>
       <xacro:insert_block name="origin_DEP" />
-      <axis xyz="0 0 1"/>
+      <axis xyz="0 0 ${driving_direction}"/>
       <dynamics damping="${damping}" friction="${friction}"/>
     </joint>
@@ -151,5 +152,5 @@
       <limit effort="${limit_drive_effort}" velocity="${limit_drive_velocity}"/>
       <origin xyz="0 0 ${-size_link / 2 - 1.1 * wheel_radius}" rpy="-1.57 0 0"/>
-      <axis xyz="0 0 1"/>
+      <axis xyz="0 0 ${driving_direction}"/>
       <dynamics damping="${damping}" friction="${friction}"/>
     </joint>
@@ -203,9 +204,9 @@
     <origin xyz="0.3 ${size_base / 2} 0" rpy="${- pi / 2} 0 0"/>
   </xacro:boogie>
-  <xacro:wheel_assembly position="LF" boogie_name="${side_boogie_left_name}">
+  <xacro:wheel_assembly position="LF" boogie_name="${side_boogie_left_name}" driving_direction="1">
     <origin xyz="0.2 0 0.05" rpy="0 0 0"/>
     <origin xyz="0.1 0 0.1" rpy="${pi / 2} 0 0"/>
   </xacro:wheel_assembly>
-  <xacro:wheel_assembly position="LM" boogie_name="${side_boogie_left_name}">
+  <xacro:wheel_assembly position="LM" boogie_name="${side_boogie_left_name}" driving_direction="1">
     <origin xyz="-0.2 0 0.05" rpy="0 0 0"/>
     <origin xyz="-0.1 0 0.1" rpy="${pi / 2} 0 0"/>
@@ -216,9 +217,9 @@
     <origin xyz="0.3 -${size_base / 2} 0" rpy="${- pi / 2} 0 ${pi}"/>
   </xacro:boogie>
-  <xacro:wheel_assembly position="RF" boogie_name="${side_boogie_right_name}">
+  <xacro:wheel_assembly position="RF" boogie_name="${side_boogie_right_name}" driving_direction="-1">
     <origin xyz="-0.2 0 0.05" rpy="0 0 0"/>
     <origin xyz="-0.1 0 0.1" rpy="${pi / 2} 0 0"/>
   </xacro:wheel_assembly>
-  <xacro:wheel_assembly position="RM" boogie_name="${side_boogie_right_name}">
+  <xacro:wheel_assembly position="RM" boogie_name="${side_boogie_right_name}" driving_direction="-1">
     <origin xyz="0.2 0 0.05" rpy="0 0 0"/>
     <origin xyz="0.1 0 0.1" rpy="${pi / 2} 0 0"/>
@@ -229,11 +230,11 @@
     <origin xyz="-${size_base / 2 + 0.05} 0 0" rpy="${- pi / 2} 0 ${pi / 2}"/>
   </xacro:boogie>
-  <xacro:wheel_assembly position="RR" boogie_name="${side_boogie_rear_name}">
+  <xacro:wheel_assembly position="LR" boogie_name="${side_boogie_rear_name}" driving_direction="1">
+    <origin xyz="0.3 0 0.05" rpy="0 ${pi / 2} 0"/>
+    <origin xyz="-0.1 0 0.1" rpy="${pi / 2} 0 0"/>
+  </xacro:wheel_assembly>
+  <xacro:wheel_assembly position="RR" boogie_name="${side_boogie_rear_name}" driving_direction="-1">
     <origin xyz="-0.3 0 0.05" rpy="0 ${3 * pi / 2} 0"/>
     <origin xyz="0.1 0 0.1" rpy="${pi / 2} 0 0"/>
   </xacro:wheel_assembly>
-  <xacro:wheel_assembly position="LR" boogie_name="${side_boogie_rear_name}">
-    <origin xyz="0.3 0 0.05" rpy="0 ${pi / 2} 0"/>
-    <origin xyz="-0.1 0 0.1" rpy="${pi / 2} 0 0"/>
-  </xacro:wheel_assembly>
 </robot>

Commit message: set steering limit to 100 deg

File: urdf/marta.xacro (robot description, xacro)
@@ -12,6 +12,6 @@
   <xacro:property name="limit_drive_velocity" value="1.0" />
   <xacro:property name="limit_steer_effort" value="100.0" />
-  <xacro:property name="limit_steer_lower" value="${-pi / 2}" />
-  <xacro:property name="limit_steer_upper" value="${pi / 2}" />
+  <xacro:property name="limit_steer_lower" value="${-100*pi/180}" />
+  <xacro:property name="limit_steer_upper" value="${ 100*pi/180}" />
   <xacro:property name="limit_steer_velocity" value="1.0" />
   <xacro:property name="side_boogie_lower" value="${-pi / 4}" />
