Commit message: half working version. Link definitions are offset, PID 0controlls are shitty and mass is way too high as otherwise the inertia is too low

File: urdf/marta.xacro (robot description, xacro)
@@ -1,9 +1,7 @@
 <?xml version="1.0"?>
 <robot name="marta" xmlns:xacro="http://www.ros.org/wiki/xacro">
+  <!-- PHYSICS -->
   <xacro:property name="damping" value="0.1" />
   <xacro:property name="friction" value="0.1" />
-  <xacro:property name="size_base" value="0.5" />
-  <xacro:property name="size_link" value="0.06" />
-  <xacro:property name="mass" value="1.0" />
   <!-- CHASSIS -->
   <xacro:property name="chassis_mass" value="10.0" />
@@ -12,5 +10,6 @@
   <xacro:property name="chassis_z" value="0.343" />
   <!-- SIDE BOGIE -->
-  <xacro:property name="side_bogie_mass" value="0.15" />
+  <!-- <xacro:property name="side_bogie_mass" value="0.15" /> -->
+  <xacro:property name="side_bogie_mass" value="1.5" />
   <xacro:property name="side_bogie_l" value="0.26" />
   <xacro:property name="side_bogie_r" value="0.0125" />
@@ -19,5 +18,6 @@
   <xacro:property name="side_bogie_pos_z" value="-0.015" />
   <!-- REAR BOGIE -->
-  <xacro:property name="rear_bogie_mass" value="0.4" />
+  <!-- <xacro:property name="rear_bogie_mass" value="0.4" /> -->
+  <xacro:property name="rear_bogie_mass" value="4" />
   <xacro:property name="rear_bogie_l" value="0.559" />
   <xacro:property name="rear_bogie_r" value="0.0125" />
@@ -26,5 +26,6 @@
   <xacro:property name="rear_bogie_pos_z" value="-0.015" />
   <!-- DEPLOYMENT JOINT -->
-  <xacro:property name="dep_mass" value="0.57" />
+  <!-- <xacro:property name="dep_mass" value="0.57" /> -->
+  <xacro:property name="dep_mass" value="5.7" />
   <xacro:property name="dep_x" value="0.056" />
   <xacro:property name="dep_y" value="0.088" />
@@ -38,14 +39,17 @@
   <xacro:property name="rear_dep_pos_z" value="0.0325" />
   <!-- STEERING JOINT -->
-  <xacro:property name="str_mass" value="0.025" />
+  <!-- <xacro:property name="str_mass" value="0.025" /> -->
+  <xacro:property name="str_mass" value="0.25" />
   <xacro:property name="str_x" value="0.079" />
   <xacro:property name="str_y" value="0.0435" />
   <xacro:property name="str_z" value="0.1015" />
   <xacro:property name="str_pos_short_x" value="0.02" />
+  <xacro:property name="test" value="0.02" />
   <xacro:property name="str_pos_long_x" value="0.045" />
   <xacro:property name="str_pos_y" value="0.031" />
   <xacro:property name="str_pos_z" value="0.0305" />
   <!-- WHEEL -->
-  <xacro:property name="wheel_mass" value="0.23" />
+  <!-- <xacro:property name="wheel_mass" value="0.23" /> -->
+  <xacro:property name="wheel_mass" value="2.3" />
   <xacro:property name="wheel_x" value="0.0" />
   <xacro:property name="wheel_y" value="0.0" />
@@ -54,7 +58,7 @@
   <xacro:property name="wheel_r" value="${0.1425 / 2}" />
   <!-- DRIVE LIMITS -->
-  <xacro:property name="limit_drive_effort" value="100.0" />
+  <xacro:property name="limit_drive_effort" value="1000.0" />
   <xacro:property name="limit_drive_velocity" value="1.0" />
-  <xacro:property name="limit_steer_effort" value="100.0" />
+  <xacro:property name="limit_steer_effort" value="1000.0" />
   <xacro:property name="limit_steer_lower" value="${-100*pi/180}" />
   <xacro:property name="limit_steer_upper" value="${ 100*pi/180}" />
@@ -65,5 +69,5 @@
   <!-- Import all Gazebo-customization elements, including Gazebo colors and plugins -->
   <xacro:include filename="$(find rover_config)/urdf/marta.gazebo" />
-  <!-- Base of the rover, must be named "base_link" -->
+  <!-- CHASSIS DEFINITION (must be called base_link)-->
   <link name="base_link">
     <collision>
@@ -90,5 +94,5 @@
     </visual>
   </link>
-  <!-- Definition for a side bogie assembly -->
+  <!-- BOGIE DEFINITION -->
   <xacro:macro name="bogie" params="position bogie_mass bogie_r bogie_l *origin_bogie *geometry">
     <xacro:property name="bogie_link" value="link_bogie_${position}" />
@@ -104,4 +108,5 @@
         <origin xyz="0 0 0" rpy="0 ${pi / 2} 0"/>
         <geometry>
+          <!-- <cylinder length="0.01" radius="0.01"/> -->
           <xacro:insert_block name="geometry" />
         </geometry>
@@ -167,5 +172,4 @@
       <child link="link_STR_${position}"/>
       <limit effort="${limit_steer_effort}" lower="${limit_steer_lower}" upper="${limit_steer_upper}" velocity="${limit_steer_velocity}"/>
-      <!-- <origin xyz="0.15 0 0.15" rpy="${pi / 2} 0 0"/> -->
       <xacro:insert_block name="origin_STR" />
       <axis xyz="0 0 1"/>
@@ -270,13 +274,9 @@
   </xacro:bogie>
   <xacro:wheel_assembly position="LF" bogie_name="${side_bogie_left_name}" driving_direction="1">
-    <!-- origin_DEP -->
     <origin xyz="${side_dep_pos_front_x} ${side_dep_pos_y} ${side_dep_pos_z}" rpy="0 0 0"/>
-    <!-- origin_STR -->
     <origin xyz="${str_pos_short_x} ${str_pos_y} ${str_pos_z}" rpy="${pi / 2} 0 0"/>
   </xacro:wheel_assembly>
   <xacro:wheel_assembly position="LM" bogie_name="${side_bogie_left_name}" driving_direction="1">
-    <!-- origin_DEP -->
     <origin xyz="-${side_dep_pos_mid_x} ${side_dep_pos_y} ${side_dep_pos_z}" rpy="0 0 0"/>
-    <!-- origin_STR -->
     <origin xyz="-${str_pos_long_x} ${str_pos_y} ${str_pos_z}" rpy="${pi / 2} 0 0"/>
   </xacro:wheel_assembly>
@@ -288,13 +288,9 @@
   </xacro:bogie>
   <xacro:wheel_assembly position="RF" bogie_name="${side_bogie_right_name}" driving_direction="-1">
-    <!-- origin_DEP -->
     <origin xyz="-${side_dep_pos_front_x} ${side_dep_pos_y} ${side_dep_pos_z}" rpy="0 0 0"/>
-    <!-- origin_STR -->
     <origin xyz="-${str_pos_short_x} ${str_pos_y} ${str_pos_z}" rpy="${pi / 2} 0 0"/>
   </xacro:wheel_assembly>
   <xacro:wheel_assembly position="RM" bogie_name="${side_bogie_right_name}" driving_direction="-1">
-    <!-- origin_DEP -->
     <origin xyz="${side_dep_pos_mid_x} ${side_dep_pos_y} ${side_dep_pos_z}" rpy="0 0 0"/>
-    <!-- origin_STR -->
     <origin xyz="${str_pos_long_x} ${str_pos_y} ${str_pos_z}" rpy="${pi / 2} 0 0"/>
   </xacro:wheel_assembly>
@@ -306,14 +302,14 @@
   </xacro:bogie>
   <xacro:wheel_assembly position="LR" bogie_name="${side_bogie_rear_name}" driving_direction="1">
-    <!-- origin_DEP -->
     <origin xyz="${rear_dep_pos_x} ${rear_dep_pos_y} ${rear_dep_pos_z}" rpy="0 ${pi / 2} 0"/>
-    <!-- origin_STR -->
-    <origin xyz="-${str_pos_short_x} ${str_pos_y} ${str_pos_z}" rpy="${pi / 2} 0 0"/>
+    <!-- <origin xyz="0.3 0 0.05" rpy="0 ${pi / 2} 0"/> -->
+    <!-- <origin xyz="-${str_pos_short_x} ${str_pos_y} ${str_pos_z}" rpy="${pi / 2} 0 0"/> -->
+    <origin xyz="-${test} ${str_pos_y} ${str_pos_z}" rpy="${pi / 2} 0 0"/>
   </xacro:wheel_assembly>
   <xacro:wheel_assembly position="RR" bogie_name="${side_bogie_rear_name}" driving_direction="-1">
-    <!-- origin_DEP -->
     <origin xyz="-${rear_dep_pos_x} ${rear_dep_pos_y} ${rear_dep_pos_z}" rpy="0 ${3 * pi / 2} 0"/>
-    <!-- origin_STR -->
-    <origin xyz="${str_pos_short_x} ${str_pos_y} ${str_pos_z}" rpy="${pi / 2} 0 0"/>
+    <!-- <origin xyz="-0.3 0 0.05" rpy="0 ${3 * pi / 2} 0"/> -->
+    <!-- <origin xyz="${str_pos_short_x} ${str_pos_y} ${str_pos_z}" rpy="${pi / 2} 0 0"/> -->
+    <origin xyz="${test} ${str_pos_y} ${str_pos_z}" rpy="${pi / 2} 0 0"/>
   </xacro:wheel_assembly>
 </robot>

Commit message: fixed the MaRTA model by setting the solver iterations in gazebo to >100. This can be loaded from the world as whon in worlds/empty.world

File: urdf/marta.xacro (robot description, xacro)
@@ -2,5 +2,5 @@
 <robot name="marta" xmlns:xacro="http://www.ros.org/wiki/xacro">
   <!-- PHYSICS -->
-  <xacro:property name="damping" value="0.1" />
+  <xacro:property name="damping" value="2" />
   <xacro:property name="friction" value="0.1" />
   <!-- CHASSIS -->
@@ -10,4 +10,7 @@
   <xacro:property name="chassis_z" value="0.343" />
   <!-- SIDE BOGIE -->
+  <!-- TODO: FIX INTERTIA and mass. Mass
+  values were multiplied by 10 as the model exploded otherwise due to low inertia.
+  The real values are commented out.-->
   <!-- <xacro:property name="side_bogie_mass" value="0.15" /> -->
   <xacro:property name="side_bogie_mass" value="1.5" />
@@ -45,5 +48,4 @@
   <xacro:property name="str_z" value="0.1015" />
   <xacro:property name="str_pos_short_x" value="0.02" />
-  <xacro:property name="test" value="0.02" />
   <xacro:property name="str_pos_long_x" value="0.045" />
   <xacro:property name="str_pos_y" value="0.031" />
@@ -303,13 +305,9 @@
   <xacro:wheel_assembly position="LR" bogie_name="${side_bogie_rear_name}" driving_direction="1">
     <origin xyz="${rear_dep_pos_x} ${rear_dep_pos_y} ${rear_dep_pos_z}" rpy="0 ${pi / 2} 0"/>
-    <!-- <origin xyz="0.3 0 0.05" rpy="0 ${pi / 2} 0"/> -->
-    <!-- <origin xyz="-${str_pos_short_x} ${str_pos_y} ${str_pos_z}" rpy="${pi / 2} 0 0"/> -->
-    <origin xyz="-${test} ${str_pos_y} ${str_pos_z}" rpy="${pi / 2} 0 0"/>
+    <origin xyz="-${str_pos_short_x} ${str_pos_y} ${str_pos_z}" rpy="${pi / 2} 0 0"/>
   </xacro:wheel_assembly>
   <xacro:wheel_assembly position="RR" bogie_name="${side_bogie_rear_name}" driving_direction="-1">
     <origin xyz="-${rear_dep_pos_x} ${rear_dep_pos_y} ${rear_dep_pos_z}" rpy="0 ${3 * pi / 2} 0"/>
-    <!-- <origin xyz="-0.3 0 0.05" rpy="0 ${3 * pi / 2} 0"/> -->
-    <!-- <origin xyz="${str_pos_short_x} ${str_pos_y} ${str_pos_z}" rpy="${pi / 2} 0 0"/> -->
-    <origin xyz="${test} ${str_pos_y} ${str_pos_z}" rpy="${pi / 2} 0 0"/>
+    <origin xyz="${str_pos_short_x} ${str_pos_y} ${str_pos_z}" rpy="${pi / 2} 0 0"/>
   </xacro:wheel_assembly>
 </robot>

Commit message: removed testing stuff

File: urdf/marta.xacro (robot description, xacro)
@@ -110,5 +110,4 @@
         <origin xyz="0 0 0" rpy="0 ${pi / 2} 0"/>
         <geometry>
-          <!-- <cylinder length="0.01" radius="0.01"/> -->
           <xacro:insert_block name="geometry" />
         </geometry>

Commit message: fixed xacro architecture to represent real joint movement

File: urdf/marta.xacro (robot description, xacro)
@@ -13,4 +13,5 @@
   values were multiplied by 10 as the model exploded otherwise due to low inertia.
   The real values are commented out.-->
+  <!-- TODO: STR and DEP INERTIA and mass are not correct anymore  -->
   <!-- <xacro:property name="side_bogie_mass" value="0.15" /> -->
   <xacro:property name="side_bogie_mass" value="1.5" />
@@ -23,15 +24,15 @@
   <!-- <xacro:property name="rear_bogie_mass" value="0.4" /> -->
   <xacro:property name="rear_bogie_mass" value="4" />
-  <xacro:property name="rear_bogie_l" value="0.559" />
+  <xacro:property name="rear_bogie_l" value="0.5815" />
   <xacro:property name="rear_bogie_r" value="0.0125" />
   <xacro:property name="rear_bogie_pos_x" value="-0.316" />
   <xacro:property name="rear_bogie_pos_y" value="0" />
   <xacro:property name="rear_bogie_pos_z" value="-0.015" />
+  <xacro:property name="dep_x" value="0.056" />
+  <xacro:property name="dep_y" value="0.088" />
+  <xacro:property name="dep_z" value="0.0855" />
   <!-- DEPLOYMENT JOINT -->
   <!-- <xacro:property name="dep_mass" value="0.57" /> -->
   <xacro:property name="dep_mass" value="5.7" />
-  <xacro:property name="dep_x" value="0.056" />
-  <xacro:property name="dep_y" value="0.088" />
-  <xacro:property name="dep_z" value="0.0855" />
   <xacro:property name="side_dep_pos_front_x" value="0.14" />
   <xacro:property name="side_dep_pos_mid_x" value="0.12" />
@@ -41,10 +42,11 @@
   <xacro:property name="rear_dep_pos_y" value="-0.01" />
   <xacro:property name="rear_dep_pos_z" value="0.0325" />
+  <xacro:property name="str_x" value="0.079" />
+  <xacro:property name="str_y" value="0.1015" />
+  <xacro:property name="str_z" value="0.0435" />
+  <xacro:property name="str_x_link_diff" value="0.017" />
   <!-- STEERING JOINT -->
   <!-- <xacro:property name="str_mass" value="0.025" /> -->
   <xacro:property name="str_mass" value="0.25" />
-  <xacro:property name="str_x" value="0.079" />
-  <xacro:property name="str_y" value="0.0435" />
-  <xacro:property name="str_z" value="0.1015" />
   <xacro:property name="str_pos_short_x" value="0.02" />
   <xacro:property name="str_pos_long_x" value="0.045" />
@@ -97,5 +99,5 @@
   </link>
   <!-- BOGIE DEFINITION -->
-  <xacro:macro name="bogie" params="position bogie_mass bogie_r bogie_l *origin_bogie *geometry">
+  <xacro:macro name="bogie" params="position bogie_mass bogie_r bogie_l dep_pos_z dep_rot_y *origin_bogie *geometry">
     <xacro:property name="bogie_link" value="link_bogie_${position}" />
     <joint name="joint_bogie_${position}" type="revolute">
@@ -123,8 +125,34 @@
               iyz="0"/>
       </inertial>
+      <!-- BAR -->
       <visual>
         <origin xyz="0 0 0" rpy="0 ${pi / 2} 0"/>
         <geometry>
           <xacro:insert_block name="geometry" />
+        </geometry>
+      </visual>
+      <!-- DEP MOTORS -->
+      <collision>
+        <origin xyz="${bogie_l/2} -0.0325 ${dep_pos_z-dep_z/2}" rpy="0 ${dep_rot_y} 0"/>
+        <geometry>
+          <box size="${dep_x} ${dep_y} ${dep_z}"/>
+        </geometry>
+      </collision>
+      <visual>
+        <origin xyz="${bogie_l/2} -0.0325 ${dep_pos_z-dep_z/2}" rpy="0 ${dep_rot_y} 0"/>
+        <geometry>
+          <box size="${dep_x} ${dep_y} ${dep_z}"/>
+        </geometry>
+      </visual>
+      <collision>
+        <origin xyz="${-bogie_l/2} -0.0325 ${dep_pos_z-dep_z/2}" rpy="0 ${dep_rot_y} 0"/>
+        <geometry>
+          <box size="${dep_x} ${dep_y} ${dep_z}"/>
+        </geometry>
+      </collision>
+      <visual>
+        <origin xyz="${-bogie_l/2} -0.0325 ${dep_pos_z-dep_z/2}" rpy="0 ${dep_rot_y} 0"/>
+        <geometry>
+          <box size="${dep_x} ${dep_y} ${dep_z}"/>
         </geometry>
       </visual>
@@ -133,5 +161,5 @@
   <!-- Definition for a wheel assembly -->
   <!-- Driving direction is used to invert the direction of the deployment and driving joint -->
-  <xacro:macro name="wheel_assembly" params="position bogie_name driving_direction *origin_DEP *origin_STR">
+  <xacro:macro name="wheel_assembly" params="position bogie_name driving_direction str_pos_x *origin_DEP *origin_STR">
     <!-- DEPLOYMENT JOINT -->
     <joint name="joint_DEP_${position}" type="revolute">
@@ -146,9 +174,15 @@
     <link name="link_DEP_${position}">
       <collision>
-        <origin xyz="0 0 -${dep_z/2}" rpy="0 0 0"/>
-        <geometry>
-          <box size="${dep_x} ${dep_y} ${dep_z}"/>
-        </geometry>
-      </collision>
+        <origin xyz="${str_pos_x} ${str_pos_y-str_y/2} ${str_pos_z}" rpy="0 0 0"/>
+        <geometry>
+          <box size="${str_x} ${str_y} ${str_z}"/>
+        </geometry>
+      </collision>
+      <visual>
+        <origin xyz="${str_pos_x} ${str_pos_y-str_y/2} ${str_pos_z}" rpy="0 0 0"/>
+        <geometry>
+          <box size="${str_x} ${str_y} ${str_z}"/>
+        </geometry>
+      </visual>
       <inertial>
           <mass value="${dep_mass}"/>
@@ -161,10 +195,4 @@
               iyz="0"/>
       </inertial>
-      <visual>
-        <origin xyz="0 0 -${dep_z/2}" rpy="0 0 0"/>
-        <geometry>
-          <box size="${dep_x} ${dep_y} ${dep_z}"/>
-        </geometry>
-      </visual>
     </link>
     <!-- STEERING JOINT -->
@@ -179,10 +207,29 @@
     <!-- STEERING LINK -->
     <link name="link_STR_${position}">
-      <collision>
-        <origin xyz="0 0 ${str_z/2}" rpy="0 0 0"/>
-        <geometry>
-          <box size="${str_x} ${str_y} ${str_z}"/>
-        </geometry>
-      </collision>
+      <!-- Wheel bracket -->
+      <collision>
+        <origin xyz="0.0 0.049 -0.0545" rpy="0 0 0"/>
+        <geometry>
+          <box size="0.044 0.006 0.109"/>
+        </geometry>
+      </collision>
+      <visual>
+        <origin xyz="0.0 0.049 -0.0545" rpy="0 0 0"/>
+        <geometry>
+          <box size="0.044 0.006 0.109"/>
+        </geometry>
+      </visual>
+      <collision>
+        <origin xyz="0.0 0.013 -0.00325" rpy="0 0 0"/>
+        <geometry>
+          <box size="0.044 0.078 0.0065"/>
+        </geometry>
+      </collision>
+      <visual>
+        <origin xyz="0.0 0.013 -0.00325" rpy="0 0 0"/>
+        <geometry>
+          <box size="0.044 0.078 0.0065"/>
+        </geometry>
+      </visual>
       <inertial>
           <mass value="${str_mass}"/>
@@ -195,16 +242,4 @@
               iyz="0"/>
       </inertial>
-      <visual>
-        <origin xyz="0 0 ${str_z/2}" rpy="0 0 0"/>
-        <geometry>
-          <box size="${str_x} ${str_y} ${str_z}"/>
-        </geometry>
-      </visual>
-      <visual>
-        <origin xyz="0.0 0.049 -0.0545" rpy="0 0 0"/>
-        <geometry>
-          <box size="0.044 0.006 0.109"/>
-        </geometry>
-      </visual>
     </link>
     <!-- DRIVING JOINT -->
@@ -248,5 +283,5 @@
       </visual>
     </link>
-    <transmission name="_STR_${position}">
+    <transmission name="transmission_STR_${position}">
       <type>transmission_interface/SimpleTransmission</type>
       <joint name="joint_STR_${position}">
@@ -270,13 +305,13 @@
   <!-- LEFT BOGIE  -->
   <xacro:property name="side_bogie_left_name" value="LFB" />
-  <xacro:bogie position="${side_bogie_left_name}" bogie_mass="${side_bogie_mass}" bogie_r="${side_bogie_r}" bogie_l="${side_bogie_l}">
+  <xacro:bogie position="${side_bogie_left_name}" bogie_mass="${side_bogie_mass}" bogie_r="${side_bogie_r}" bogie_l="${side_bogie_l}" dep_pos_z="${side_dep_pos_z}" dep_rot_y="${0.0}">
     <origin xyz="${side_bogie_pos_x} ${side_bogie_pos_y} ${side_bogie_pos_z}" rpy="${- pi / 2} 0 0"/>
     <cylinder length="${side_bogie_l}" radius="${side_bogie_r}"/>
   </xacro:bogie>
-  <xacro:wheel_assembly position="LF" bogie_name="${side_bogie_left_name}" driving_direction="1">
+  <xacro:wheel_assembly position="LF" bogie_name="${side_bogie_left_name}" driving_direction="1" str_pos_x="${str_pos_short_x-str_x_link_diff}">
     <origin xyz="${side_dep_pos_front_x} ${side_dep_pos_y} ${side_dep_pos_z}" rpy="0 0 0"/>
     <origin xyz="${str_pos_short_x} ${str_pos_y} ${str_pos_z}" rpy="${pi / 2} 0 0"/>
   </xacro:wheel_assembly>
-  <xacro:wheel_assembly position="LM" bogie_name="${side_bogie_left_name}" driving_direction="1">
+  <xacro:wheel_assembly position="LM" bogie_name="${side_bogie_left_name}" driving_direction="1" str_pos_x="${-(str_pos_long_x-str_x_link_diff)}">
     <origin xyz="-${side_dep_pos_mid_x} ${side_dep_pos_y} ${side_dep_pos_z}" rpy="0 0 0"/>
     <origin xyz="-${str_pos_long_x} ${str_pos_y} ${str_pos_z}" rpy="${pi / 2} 0 0"/>
@@ -284,13 +319,13 @@
   <!-- RIGHT BOGIE  -->
   <xacro:property name="side_bogie_right_name" value="RFB" />
-  <xacro:bogie position="${side_bogie_right_name}" bogie_mass="${side_bogie_mass}" bogie_r="${side_bogie_r}" bogie_l="${side_bogie_l}">
+  <xacro:bogie position="${side_bogie_right_name}" bogie_mass="${side_bogie_mass}" bogie_r="${side_bogie_r}" bogie_l="${side_bogie_l}" dep_pos_z="${side_dep_pos_z}" dep_rot_y="${0.0}">
     <origin xyz="${side_bogie_pos_x} -${side_bogie_pos_y} ${side_bogie_pos_z}" rpy="${- pi / 2} 0 ${pi}"/>
     <cylinder length="${side_bogie_l}" radius="${side_bogie_r}"/>
   </xacro:bogie>
-  <xacro:wheel_assembly position="RF" bogie_name="${side_bogie_right_name}" driving_direction="-1">
+  <xacro:wheel_assembly position="RF" bogie_name="${side_bogie_right_name}" driving_direction="-1" str_pos_x="${-(str_pos_short_x-str_x_link_diff)}">
     <origin xyz="-${side_dep_pos_front_x} ${side_dep_pos_y} ${side_dep_pos_z}" rpy="0 0 0"/>
     <origin xyz="-${str_pos_short_x} ${str_pos_y} ${str_pos_z}" rpy="${pi / 2} 0 0"/>
   </xacro:wheel_assembly>
-  <xacro:wheel_assembly position="RM" bogie_name="${side_bogie_right_name}" driving_direction="-1">
+  <xacro:wheel_assembly position="RM" bogie_name="${side_bogie_right_name}" driving_direction="-1" str_pos_x="${(str_pos_long_x-str_x_link_diff)}">
     <origin xyz="${side_dep_pos_mid_x} ${side_dep_pos_y} ${side_dep_pos_z}" rpy="0 0 0"/>
     <origin xyz="${str_pos_long_x} ${str_pos_y} ${str_pos_z}" rpy="${pi / 2} 0 0"/>
@@ -298,13 +333,13 @@
   <!-- REAR BOGIE  -->
   <xacro:property name="side_bogie_rear_name" value="MRB" />
-  <xacro:bogie position="${side_bogie_rear_name}" bogie_mass="${rear_bogie_mass}" bogie_r="${rear_bogie_r}" bogie_l="${rear_bogie_l}">
+  <xacro:bogie position="${side_bogie_rear_name}" bogie_mass="${rear_bogie_mass}" bogie_r="${rear_bogie_r}" bogie_l="${rear_bogie_l}" dep_pos_z="${rear_dep_pos_z}" dep_rot_y="${-pi/2}">
     <origin xyz="${rear_bogie_pos_x} ${rear_bogie_pos_y} ${rear_bogie_pos_z}" rpy="${- pi / 2} 0 ${pi / 2}"/>
     <cylinder length="${rear_bogie_l}" radius="${rear_bogie_r}"/>
   </xacro:bogie>
-  <xacro:wheel_assembly position="LR" bogie_name="${side_bogie_rear_name}" driving_direction="1">
+  <xacro:wheel_assembly position="LR" bogie_name="${side_bogie_rear_name}" driving_direction="1" str_pos_x="${-(str_pos_short_x-str_x_link_diff)}">
     <origin xyz="${rear_dep_pos_x} ${rear_dep_pos_y} ${rear_dep_pos_z}" rpy="0 ${pi / 2} 0"/>
     <origin xyz="-${str_pos_short_x} ${str_pos_y} ${str_pos_z}" rpy="${pi / 2} 0 0"/>
   </xacro:wheel_assembly>
-  <xacro:wheel_assembly position="RR" bogie_name="${side_bogie_rear_name}" driving_direction="-1">
+  <xacro:wheel_assembly position="RR" bogie_name="${side_bogie_rear_name}" driving_direction="-1" str_pos_x="${(str_pos_short_x-str_x_link_diff)}">
     <origin xyz="-${rear_dep_pos_x} ${rear_dep_pos_y} ${rear_dep_pos_z}" rpy="0 ${3 * pi / 2} 0"/>
     <origin xyz="${str_pos_short_x} ${str_pos_y} ${str_pos_z}" rpy="${pi / 2} 0 0"/>
