Commit message: fixed rear bogie deployment motor positions

File: urdf/marta.xacro (robot description, xacro)
@@ -109,10 +109,4 @@
     </joint>
     <link name="link_bogie_${position}">
-      <collision>
-        <origin xyz="0 0 0" rpy="0 ${pi / 2} 0"/>
-        <geometry>
-          <xacro:insert_block name="geometry" />
-        </geometry>
-      </collision>
       <inertial>
         <mass value="${bogie_mass}"/>
@@ -126,13 +120,19 @@
       </inertial>
       <!-- BAR -->
-      <visual>
+      <collision>
         <origin xyz="0 0 0" rpy="0 ${pi / 2} 0"/>
         <geometry>
           <xacro:insert_block name="geometry" />
         </geometry>
-      </visual>
-      <!-- DEP MOTORS -->
-      <collision>
-        <origin xyz="${bogie_l/2} -0.0325 ${dep_pos_z-dep_z/2}" rpy="0 ${dep_rot_y} 0"/>
+      </collision>
+      <visual>
+        <origin xyz="0 0 0" rpy="0 ${pi / 2} 0"/>
+        <geometry>
+          <xacro:insert_block name="geometry" />
+        </geometry>
+      </visual>
+      <!-- DEPLOYMENT MOTORS -->
+      <collision>
+        <origin xyz="${bogie_l/2} -0.0325 ${dep_pos_z}" rpy="0 ${dep_rot_y} 0"/>
         <geometry>
           <box size="${dep_x} ${dep_y} ${dep_z}"/>
@@ -140,5 +140,5 @@
       </collision>
       <visual>
-        <origin xyz="${bogie_l/2} -0.0325 ${dep_pos_z-dep_z/2}" rpy="0 ${dep_rot_y} 0"/>
+        <origin xyz="${bogie_l/2} -0.0325 ${dep_pos_z}" rpy="0 ${dep_rot_y} 0"/>
         <geometry>
           <box size="${dep_x} ${dep_y} ${dep_z}"/>
@@ -146,5 +146,5 @@
       </visual>
       <collision>
-        <origin xyz="${-bogie_l/2} -0.0325 ${dep_pos_z-dep_z/2}" rpy="0 ${dep_rot_y} 0"/>
+        <origin xyz="${-bogie_l/2} -0.0325 ${dep_pos_z}" rpy="0 ${dep_rot_y} 0"/>
         <geometry>
           <box size="${dep_x} ${dep_y} ${dep_z}"/>
@@ -152,5 +152,5 @@
       </collision>
       <visual>
-        <origin xyz="${-bogie_l/2} -0.0325 ${dep_pos_z-dep_z/2}" rpy="0 ${dep_rot_y} 0"/>
+        <origin xyz="${-bogie_l/2} -0.0325 ${dep_pos_z}" rpy="0 ${dep_rot_y} 0"/>
         <geometry>
           <box size="${dep_x} ${dep_y} ${dep_z}"/>
@@ -173,16 +173,4 @@
     <!-- DEPLOYMENT LINK-->
     <link name="link_DEP_${position}">
-      <collision>
-        <origin xyz="${str_pos_x} ${str_pos_y-str_y/2} ${str_pos_z}" rpy="0 0 0"/>
-        <geometry>
-          <box size="${str_x} ${str_y} ${str_z}"/>
-        </geometry>
-      </collision>
-      <visual>
-        <origin xyz="${str_pos_x} ${str_pos_y-str_y/2} ${str_pos_z}" rpy="0 0 0"/>
-        <geometry>
-          <box size="${str_x} ${str_y} ${str_z}"/>
-        </geometry>
-      </visual>
       <inertial>
           <mass value="${dep_mass}"/>
@@ -195,4 +183,17 @@
               iyz="0"/>
       </inertial>
+      <!-- STEERING MOTOR -->
+      <collision>
+        <origin xyz="${str_pos_x} ${str_pos_y-str_y/2} ${str_pos_z}" rpy="0 0 0"/>
+        <geometry>
+          <box size="${str_x} ${str_y} ${str_z}"/>
+        </geometry>
+      </collision>
+      <visual>
+        <origin xyz="${str_pos_x} ${str_pos_y-str_y/2} ${str_pos_z}" rpy="0 0 0"/>
+        <geometry>
+          <box size="${str_x} ${str_y} ${str_z}"/>
+        </geometry>
+      </visual>
     </link>
     <!-- STEERING JOINT -->
@@ -207,29 +208,4 @@
     <!-- STEERING LINK -->
     <link name="link_STR_${position}">
-      <!-- Wheel bracket -->
-      <collision>
-        <origin xyz="0.0 0.049 -0.0545" rpy="0 0 0"/>
-        <geometry>
-          <box size="0.044 0.006 0.109"/>
-        </geometry>
-      </collision>
-      <visual>
-        <origin xyz="0.0 0.049 -0.0545" rpy="0 0 0"/>
-        <geometry>
-          <box size="0.044 0.006 0.109"/>
-        </geometry>
-      </visual>
-      <collision>
-        <origin xyz="0.0 0.013 -0.00325" rpy="0 0 0"/>
-        <geometry>
-          <box size="0.044 0.078 0.0065"/>
-        </geometry>
-      </collision>
-      <visual>
-        <origin xyz="0.0 0.013 -0.00325" rpy="0 0 0"/>
-        <geometry>
-          <box size="0.044 0.078 0.0065"/>
-        </geometry>
-      </visual>
       <inertial>
           <mass value="${str_mass}"/>
@@ -242,4 +218,29 @@
               iyz="0"/>
       </inertial>
+      <!-- WHEEL BRACKET -->
+      <collision>
+        <origin xyz="0.0 0.049 -0.0545" rpy="0 0 0"/>
+        <geometry>
+          <box size="0.044 0.006 0.109"/>
+        </geometry>
+      </collision>
+      <visual>
+        <origin xyz="0.0 0.049 -0.0545" rpy="0 0 0"/>
+        <geometry>
+          <box size="0.044 0.006 0.109"/>
+        </geometry>
+      </visual>
+      <collision>
+        <origin xyz="0.0 0.013 -0.00325" rpy="0 0 0"/>
+        <geometry>
+          <box size="0.044 0.078 0.0065"/>
+        </geometry>
+      </collision>
+      <visual>
+        <origin xyz="0.0 0.013 -0.00325" rpy="0 0 0"/>
+        <geometry>
+          <box size="0.044 0.078 0.0065"/>
+        </geometry>
+      </visual>
     </link>
     <!-- DRIVING JOINT -->
@@ -305,5 +306,5 @@
   <!-- LEFT BOGIE  -->
   <xacro:property name="side_bogie_left_name" value="LFB" />
-  <xacro:bogie position="${side_bogie_left_name}" bogie_mass="${side_bogie_mass}" bogie_r="${side_bogie_r}" bogie_l="${side_bogie_l}" dep_pos_z="${side_dep_pos_z}" dep_rot_y="${0.0}">
+  <xacro:bogie position="${side_bogie_left_name}" bogie_mass="${side_bogie_mass}" bogie_r="${side_bogie_r}" bogie_l="${side_bogie_l}" dep_pos_z="${side_dep_pos_z-dep_z/2}" dep_rot_y="${0.0}">
     <origin xyz="${side_bogie_pos_x} ${side_bogie_pos_y} ${side_bogie_pos_z}" rpy="${- pi / 2} 0 0"/>
     <cylinder length="${side_bogie_l}" radius="${side_bogie_r}"/>
@@ -319,5 +320,5 @@
   <!-- RIGHT BOGIE  -->
   <xacro:property name="side_bogie_right_name" value="RFB" />
-  <xacro:bogie position="${side_bogie_right_name}" bogie_mass="${side_bogie_mass}" bogie_r="${side_bogie_r}" bogie_l="${side_bogie_l}" dep_pos_z="${side_dep_pos_z}" dep_rot_y="${0.0}">
+  <xacro:bogie position="${side_bogie_right_name}" bogie_mass="${side_bogie_mass}" bogie_r="${side_bogie_r}" bogie_l="${side_bogie_l}" dep_pos_z="${side_dep_pos_z-dep_z/2}" dep_rot_y="${0.0}">
     <origin xyz="${side_bogie_pos_x} -${side_bogie_pos_y} ${side_bogie_pos_z}" rpy="${- pi / 2} 0 ${pi}"/>
     <cylinder length="${side_bogie_l}" radius="${side_bogie_r}"/>

Commit message: added additional collision bodies to wheel

File: urdf/marta.xacro (robot description, xacro)
@@ -23,5 +23,5 @@
   <!-- REAR BOGIE -->
   <!-- <xacro:property name="rear_bogie_mass" value="0.4" /> -->
-  <xacro:property name="rear_bogie_mass" value="4" />
+  <xacro:property name="rear_bogie_mass" value="4.0" />
   <xacro:property name="rear_bogie_l" value="0.5815" />
   <xacro:property name="rear_bogie_r" value="0.0125" />
@@ -283,4 +283,10 @@
         </geometry>
       </visual>
+      <collision>
+        <origin xyz="0 0 0" rpy="0 0 0"/>
+        <geometry>
+          <cylinder length="0.104" radius="0.0255"/>
+        </geometry>
+      </collision>
     </link>
     <transmission name="transmission_STR_${position}">

Commit message: started PTU model

File: urdf/marta.xacro (robot description, xacro)
@@ -352,3 +352,8 @@
     <origin xyz="${str_pos_short_x} ${str_pos_y} ${str_pos_z}" rpy="${pi / 2} 0 0"/>
   </xacro:wheel_assembly>
+  <!-- Sensors -->
+  <xacro:include filename="$(find rover_config)/urdf/ptu.xacro" />
+  <xacro:ptu parent_link="base_link">
+    <origin xyz="0.25 0.0 0.0" rpy="0.0 0.0 0.0"/>
+  </xacro:ptu>
 </robot>

Commit message: Add Lidar sensor to MARTA rover description
- Add link and joint in xacro
- Add sensor and plugin in gazebo file

File: urdf/marta.xacro (robot description, xacro)
@@ -98,4 +98,18 @@
     </visual>
   </link>
+  <!-- LIDAR SENSOR DEFINITION -->
+  <joint name="joint_lidar" type="fixed">
+    <parent link="base_link"/>
+    <child link="lidar_link"/>
+    <origin xyz="0 0  ${chassis_z}"/>
+  </joint>
+  <link name="lidar_link">
+    <visual>
+      <origin xyz="0 0 0" rpy="0 0 0"/>
+      <geometry>
+        <box size="0.1 0.1 0.1"/>
+      </geometry>
+    </visual>
+  </link>
   <!-- BOGIE DEFINITION -->
   <xacro:macro name="bogie" params="position bogie_mass bogie_r bogie_l dep_pos_z dep_rot_y *origin_bogie *geometry">

Commit message: Put Lidar gazebo description in seperate files

File: urdf/marta.xacro (robot description, xacro)
@@ -98,18 +98,4 @@
     </visual>
   </link>
-  <!-- LIDAR SENSOR DEFINITION -->
-  <joint name="joint_lidar" type="fixed">
-    <parent link="base_link"/>
-    <child link="lidar_link"/>
-    <origin xyz="0 0  ${chassis_z}"/>
-  </joint>
-  <link name="lidar_link">
-    <visual>
-      <origin xyz="0 0 0" rpy="0 0 0"/>
-      <geometry>
-        <box size="0.1 0.1 0.1"/>
-      </geometry>
-    </visual>
-  </link>
   <!-- BOGIE DEFINITION -->
   <xacro:macro name="bogie" params="position bogie_mass bogie_r bogie_l dep_pos_z dep_rot_y *origin_bogie *geometry">
@@ -366,3 +352,8 @@
     <origin xyz="${str_pos_short_x} ${str_pos_y} ${str_pos_z}" rpy="${pi / 2} 0 0"/>
   </xacro:wheel_assembly>
+  <!-- Sensors -->
+  <xacro:include filename="$(find rover_config)/urdf/lidar.xacro"/>
+  <xacro:lidar parent_link="base_link">
+    <origin xyz="0 0  ${chassis_z}"/>
+  </xacro:lidar>
 </robot>

Commit message: added imu

File: urdf/marta.xacro (robot description, xacro)
@@ -353,7 +353,13 @@
   </xacro:wheel_assembly>
   <!-- Sensors -->
+  <!-- LIDAR -->
   <xacro:include filename="$(find rover_config)/urdf/lidar.xacro"/>
   <xacro:lidar parent_link="base_link">
     <origin xyz="0 0  ${chassis_z}"/>
   </xacro:lidar>
+  <!-- IMU -->
+  <xacro:include filename="$(find rover_config)/urdf/imu.xacro"/>
+  <xacro:imu parent_link="base_link">
+    <origin xyz="-0.2 0  0"/>
+  </xacro:imu>
 </robot>

Commit message: added options for the usage of sensors.

File: urdf/marta.xacro (robot description, xacro)
@@ -1,4 +1,7 @@
 <?xml version="1.0"?>
 <robot name="marta" xmlns:xacro="http://www.ros.org/wiki/xacro">
+  <!-- SENSOR CONFIGURATION -->
+  <xacro:property name="use_lidar" value="true" />
+  <xacro:property name="use_imu" value="true" />
   <!-- PHYSICS -->
   <xacro:property name="damping" value="2" />
@@ -354,12 +357,16 @@
   <!-- Sensors -->
   <!-- LIDAR -->
-  <xacro:include filename="$(find rover_config)/urdf/lidar.xacro"/>
-  <xacro:lidar parent_link="base_link">
-    <origin xyz="0 0  ${chassis_z}"/>
-  </xacro:lidar>
+  <xacro:if value="${use_lidar}">
+    <xacro:include filename="$(find rover_config)/urdf/lidar.xacro"/>
+    <xacro:lidar parent_link="base_link">
+      <origin xyz="0 0  ${chassis_z}"/>
+    </xacro:lidar>
+  </xacro:if>
   <!-- IMU -->
-  <xacro:include filename="$(find rover_config)/urdf/imu.xacro"/>
-  <xacro:imu parent_link="base_link">
-    <origin xyz="-0.2 0  0"/>
-  </xacro:imu>
+  <xacro:if value="${use_imu}">
+    <xacro:include filename="$(find rover_config)/urdf/imu.xacro"/>
+    <xacro:imu parent_link="base_link">
+      <origin xyz="-0.2 0  0"/>
+    </xacro:imu>
+  </xacro:if>
 </robot>

Commit message: renamed IMU to stim300, updated visuals

File: urdf/marta.xacro (robot description, xacro)
@@ -360,12 +360,12 @@
     <xacro:include filename="$(find rover_config)/urdf/lidar.xacro"/>
     <xacro:lidar parent_link="base_link">
-      <origin xyz="0 0  ${chassis_z}"/>
+      <origin xyz="0 0 ${chassis_z}"/>
     </xacro:lidar>
   </xacro:if>
   <!-- IMU -->
   <xacro:if value="${use_imu}">
-    <xacro:include filename="$(find rover_config)/urdf/imu.xacro"/>
+    <xacro:include filename="$(find rover_config)/urdf/stim300.xacro"/>
     <xacro:imu parent_link="base_link">
-      <origin xyz="-0.2 0  0"/>
+      <origin xyz="0.09 0  0"/>
     </xacro:imu>
   </xacro:if>

File: urdf/stim300.xacro (robot description, xacro)
@@ -2,5 +2,5 @@
 <robot xmlns:xacro="http://wiki.ros.org/xacro">
   <xacro:macro name="imu" params="parent_link *origin">
-    <xacro:include filename="$(find rover_config)/urdf/imu.gazebo" />
+    <xacro:include filename="$(find rover_config)/urdf/stim300.gazebo" />
     <joint name="joint_imu" type="fixed">
       <parent link="${parent_link}"/>
@@ -8,9 +8,10 @@
       <xacro:insert_block name="origin" />
     </joint>
+    <!-- STIM300 Visual -->
     <link name="link_imu">
       <visual>
         <origin xyz="0 0 0" rpy="0 0 0"/>
         <geometry>
-          <box size="0.05 0.03 0.03"/>
+          <box size="0.0386 0.0448 0.0215"/>
         </geometry>
       </visual>

Commit message: renamed lidar to specific velodyne model (vlp-16), changed 3D model to be cylindrical instead of a box.

File: urdf/marta.xacro (robot description, xacro)
@@ -353,7 +353,7 @@
   </xacro:wheel_assembly>
   <!-- Sensors -->
-  <xacro:include filename="$(find rover_config)/urdf/lidar.xacro"/>
+  <xacro:include filename="$(find rover_config)/urdf/vlp_16.xacro"/>
   <xacro:lidar parent_link="base_link">
-    <origin xyz="0 0  ${chassis_z}"/>
+    <origin xyz="0 0  ${chassis_z + 0.006}"/>
   </xacro:lidar>
 </robot>

File: urdf/vlp_16.xacro (robot description, xacro)
@@ -2,5 +2,5 @@
 <robot xmlns:xacro="http://wiki.ros.org/xacro">
   <xacro:macro name="lidar" params="parent_link *origin">
-    <xacro:include filename="$(find rover_config)/urdf/lidar.gazebo" />
+    <xacro:include filename="$(find rover_config)/urdf/vlp_16.gazebo" />
     <joint name="joint_lidar" type="fixed">
       <parent link="${parent_link}"/>
@@ -8,9 +8,16 @@
       <xacro:insert_block name="origin" />
     </joint>
+    <!-- Model of Velodyne VLP-16 LiDAR -->
     <link name="link_lidar">
       <visual>
         <origin xyz="0 0 0" rpy="0 0 0"/>
         <geometry>
-          <box size="0.1 0.1 0.1"/>
+          <cylinder length="0.0717" radius="0.05165"/>
+        </geometry>
+      </visual>
+      <visual>
+        <origin xyz="0 0 0" rpy="0 0 0"/>
+        <geometry>
+          <cylinder length="0.0717" radius="0.05165"/>
         </geometry>
       </visual>

Commit message: added gnss sensor

File: urdf/marta.xacro (robot description, xacro)
@@ -1,4 +1,5 @@
 <?xml version="1.0"?>
 <robot name="marta" xmlns:xacro="http://www.ros.org/wiki/xacro">
+  <xacro:property name="use_gnss" value="true" />
   <!-- PHYSICS -->
   <xacro:property name="damping" value="2" />
@@ -357,3 +358,10 @@
     <origin xyz="0 0  ${chassis_z}"/>
   </xacro:lidar>
+  <!-- GNSS -->
+  <xacro:if value="${use_gnss}">
+    <xacro:include filename="$(find rover_config)/urdf/gnss.xacro"/>
+    <xacro:gnss parent_link="base_link">
+      <origin xyz="0.0 0.15  ${chassis_z-0.02}"/>
+    </xacro:gnss>
+  </xacro:if>
 </robot>

Commit message: fixed framerate andadded visualize option

File: urdf/marta.xacro (robot description, xacro)
@@ -2,8 +2,8 @@
 <robot name="marta" xmlns:xacro="http://www.ros.org/wiki/xacro">
   <!-- SENSOR CONFIGURATION -->
-  <xacro:property name="use_lidar" value="true" />
-  <xacro:property name="use_imu" value="true" />
-  <xacro:property name="use_gnss" value="true" />
-  <xacro:property name="use_ptu" value="true" />
+  <xacro:property name="use_lidar" value="false" />
+  <xacro:property name="use_imu" value="false" />
+  <xacro:property name="use_gnss" value="false" />
+  <xacro:property name="use_ptu" value="false" />
   <xacro:property name="use_loc_cam" value="true" />
   <!-- PHYSICS -->

Commit message: added new gamepadparser_parameer, added effort and velocity limits

File: urdf/marta.xacro (robot description, xacro)
@@ -5,6 +5,6 @@
   <xacro:property name="use_imu" value="false" />
   <xacro:property name="use_gnss" value="false" />
-  <xacro:property name="use_ptu" value="false" />
-  <xacro:property name="use_loc_cam" value="true" />
+  <xacro:property name="use_ptu" value="true" />
+  <xacro:property name="use_loc_cam" value="false" />
   <!-- PHYSICS -->
   <xacro:property name="damping" value="2" />

File: urdf/ptu.xacro (robot description, xacro)
@@ -6,4 +6,6 @@
     <xacro:property name="ptu_damping" value="2" />
     <xacro:property name="ptu_friction" value="0.1" />
+    <xacro:property name="max_effort" value="1000.0" />
+    <xacro:property name="max_velocity" value="1.0" />
     <!-- PARAMETERS -->
     <!-- MAST LINK -->
@@ -16,5 +18,6 @@
     <xacro:property name="joint_pan_pos_z" value="${mast_l}" />
     <!-- PAN LINK -->
-    <xacro:property name="link_pan_mass" value="0.1" />
+    <!-- <xacro:property name="link_pan_mass" value="0.1" /> -->
+    <xacro:property name="link_pan_mass" value="5" />
     <xacro:property name="link_pan_x" value="0.05" />
     <xacro:property name="link_pan_y" value="0.025" />
@@ -29,5 +32,5 @@
     <xacro:property name="joint_tilt_rot_x" value="${pi/2}" />
     <!-- TILT LINK -->
-    <xacro:property name="link_tilt_mass" value="1.0" />
+    <xacro:property name="link_tilt_mass" value="5.0" />
     <xacro:property name="link_tilt_x" value="0.022" />
     <xacro:property name="link_tilt_y" value="0.0035" />
@@ -71,9 +74,9 @@
     </link>
     <!-- PAN JOINT -->
-    <joint name="joint_PAN" type="fixed">
+    <joint name="joint_PAN" type="revolute">
       <parent link="link_mast"/>
       <child link="link_pan"/>
       <origin xyz="0 0 ${joint_pan_pos_z}" rpy="0.0 0.0 0.0"/>
-      <limit effort="0" lower="${pan_lower}" upper="${pan_upper}" velocity="0"/>
+      <limit effort="${max_effort}" lower="${pan_lower}" upper="${pan_upper}" velocity="${max_velocity}"/>
       <axis xyz="0 0 1"/>
       <dynamics damping="${ptu_damping}" friction="${ptu_friction}"/>
@@ -118,9 +121,9 @@
     </link>
     <!-- TILT JOINT -->
-    <joint name="joint_TLT" type="fixed">
+    <joint name="joint_TLT" type="revolute">
       <parent link="link_pan"/>
       <child link="link_tilt"/>
       <origin xyz="0 0 ${joint_tilt_pos_z}" rpy="${joint_tilt_rot_x} 0.0 0.0"/>
-      <limit effort="0" lower="${tilt_lower}" upper="${tilt_upper}" velocity="0"/>
+      <limit effort="${max_effort}" lower="${tilt_lower}" upper="${tilt_upper}" velocity="${max_velocity}"/>
       <axis xyz="0 0 1"/>
       <dynamics damping="${ptu_damping}" friction="${ptu_friction}"/>

Commit message: increased inertias of links to make simulation stable, reduced simulation iteration count to 100 to increase simulation speed

File: urdf/marta.xacro (robot description, xacro)
@@ -2,9 +2,9 @@
 <robot name="marta" xmlns:xacro="http://www.ros.org/wiki/xacro">
   <!-- SENSOR CONFIGURATION -->
-  <xacro:property name="use_lidar" value="false" />
-  <xacro:property name="use_imu" value="false" />
-  <xacro:property name="use_gnss" value="false" />
-  <xacro:property name="use_ptu" value="true" />
-  <xacro:property name="use_loc_cam" value="false" />
+  <xacro:property name="use_lidar"    value="true" />
+  <xacro:property name="use_imu"      value="true" />
+  <xacro:property name="use_gnss"     value="true" />
+  <xacro:property name="use_ptu"      value="true" />
+  <xacro:property name="use_loc_cam"  value="true" />
   <!-- PHYSICS -->
   <xacro:property name="damping" value="2" />
@@ -118,7 +118,7 @@
         <mass value="${bogie_mass}"/>
         <inertia
-              ixx="${bogie_mass / 12.0 * (3 * bogie_r * bogie_r + bogie_l * bogie_l)}"
+              ixx="${bogie_mass /  2.0 *  bogie_r * bogie_r}"
               iyy="${bogie_mass / 12.0 * (3 * bogie_r * bogie_r + bogie_l * bogie_l)}"
-              izz="${bogie_mass /  2.0 *  bogie_r * bogie_r}"
+              izz="${bogie_mass / 12.0 * (3 * bogie_r * bogie_r + bogie_l * bogie_l)}"
               ixy="0"
               ixz="0"

File: urdf/ptu.xacro (robot description, xacro)
@@ -32,5 +32,5 @@
     <xacro:property name="joint_tilt_rot_x" value="${pi/2}" />
     <!-- TILT LINK -->
-    <xacro:property name="link_tilt_mass" value="5.0" />
+    <xacro:property name="link_tilt_mass" value="0.1" />
     <xacro:property name="link_tilt_x" value="0.022" />
     <xacro:property name="link_tilt_y" value="0.0035" />
@@ -133,5 +133,6 @@
       <inertial>
         <mass value="${link_tilt_mass}"/>
-          <inertia
+        <!-- TODO: Real inertia value causes model to become unstable. A different physics engine might help. -->
+<!--           <inertia
               ixx="${link_tilt_mass / 12.0 * (link_tilt_y * link_tilt_z / 2)}"
               iyy="${link_tilt_mass / 12.0 * (link_tilt_x * link_tilt_z / 2)}"
@@ -140,5 +141,7 @@
               ixz="0"
               iyz="0"/>
-      </inertial>
+-->
+           <inertia ixx="0.02" ixy="0" ixz="0" iyy="0.04" iyz="0" izz="0.04"/>
+        </inertial>
       <collision>
         <origin xyz="${link_tilt_pos_x} ${link_tilt_pos_y} ${link_tilt_pos_z}" rpy="0 0 0"/>

Commit message: fix rear bogie variable name

File: urdf/marta.xacro (robot description, xacro)
@@ -350,14 +350,14 @@
   </xacro:wheel_assembly>
   <!-- REAR BOGIE  -->
-  <xacro:property name="side_bogie_rear_name" value="MRB" />
-  <xacro:bogie position="${side_bogie_rear_name}" bogie_mass="${rear_bogie_mass}" bogie_r="${rear_bogie_r}" bogie_l="${rear_bogie_l}" dep_pos_z="${rear_dep_pos_z}" dep_rot_y="${-pi/2}">
+  <xacro:property name="bogie_rear_name" value="MRB" />
+  <xacro:bogie position="${bogie_rear_name}" bogie_mass="${rear_bogie_mass}" bogie_r="${rear_bogie_r}" bogie_l="${rear_bogie_l}" dep_pos_z="${rear_dep_pos_z}" dep_rot_y="${-pi/2}">
     <origin xyz="${rear_bogie_pos_x} ${rear_bogie_pos_y} ${rear_bogie_pos_z}" rpy="${- pi / 2} 0 ${pi / 2}"/>
     <cylinder length="${rear_bogie_l}" radius="${rear_bogie_r}"/>
   </xacro:bogie>
-  <xacro:wheel_assembly position="LR" bogie_name="${side_bogie_rear_name}" driving_direction="1" str_pos_x="${-(str_pos_short_x-str_x_link_diff)}">
+  <xacro:wheel_assembly position="LR" bogie_name="${bogie_rear_name}" driving_direction="1" str_pos_x="${-(str_pos_short_x-str_x_link_diff)}">
     <origin xyz="${rear_dep_pos_x} ${rear_dep_pos_y} ${rear_dep_pos_z}" rpy="0 ${pi / 2} 0"/>
     <origin xyz="-${str_pos_short_x} ${str_pos_y} ${str_pos_z}" rpy="${pi / 2} 0 0"/>
   </xacro:wheel_assembly>
-  <xacro:wheel_assembly position="RR" bogie_name="${side_bogie_rear_name}" driving_direction="-1" str_pos_x="${(str_pos_short_x-str_x_link_diff)}">
+  <xacro:wheel_assembly position="RR" bogie_name="${bogie_rear_name}" driving_direction="-1" str_pos_x="${(str_pos_short_x-str_x_link_diff)}">
     <origin xyz="-${rear_dep_pos_x} ${rear_dep_pos_y} ${rear_dep_pos_z}" rpy="0 ${3 * pi / 2} 0"/>
     <origin xyz="${str_pos_short_x} ${str_pos_y} ${str_pos_z}" rpy="${pi / 2} 0 0"/>
