Commit message: added localization camera

File: urdf/bb2.xacro (robot description, xacro)
@@ -3,5 +3,5 @@
   <xacro:macro name="bb2" params="name parent_link *origin_cam">
     <xacro:include filename="$(find rover_config)/urdf/bb2.gazebo" />
-    <xacro:sensors cam_name="${name}" />
+    <xacro:sensors cam_name="${name}"/>
     <!-- PARAMETERS -->
     <xacro:property name="link_cam_mass" value="1.0" />
@@ -14,12 +14,12 @@
     <xacro:property name="link_cam_pos_z" value="0.0" />
     <!-- CAMERA JOINT-->
-    <joint name="camera_joint" type="fixed">
+    <joint name="joint_${name}" type="fixed">
         <parent link="${parent_link}"/>
-        <child link="link_cam"/>
+        <child link="link_${name}"/>
         <xacro:insert_block name="origin_cam" />
         <axis xyz="1 0 0" />
     </joint>
     <!-- CAMERA LINK -->
-    <link name="link_cam">
+    <link name="link_${name}">
       <inertial>
         <mass value="${link_cam_mass}"/>

File: urdf/marta.xacro (robot description, xacro)
@@ -1,4 +1,6 @@
 <?xml version="1.0"?>
 <robot name="marta" xmlns:xacro="http://www.ros.org/wiki/xacro">
+  <xacro:property name="use_ptu" value="true" />
+  <xacro:property name="use_loc_cam" value="true" />
   <!-- PHYSICS -->
   <xacro:property name="damping" value="2" />
@@ -353,8 +355,18 @@
   </xacro:wheel_assembly>
   <!-- Sensors -->
-  <xacro:include filename="$(find rover_config)/urdf/ptu.xacro" />
-  <xacro:ptu parent_link="base_link">
-    <origin xyz="0.25 0.0 0.0" rpy="0.0 0.0 0.0"/>
-  </xacro:ptu>
+  <!-- PTU w/ Navigation Cam-->
+  <xacro:if value="${use_ptu}">
+    <xacro:include filename="$(find rover_config)/urdf/ptu.xacro" />
+    <xacro:ptu parent_link="base_link">
+      <origin xyz="0.25 0.0 0.0" rpy="0.0 0.0 0.0"/>
+    </xacro:ptu>
+  </xacro:if>
+  <!-- Localization Cam -->
+  <xacro:if value="${use_loc_cam}">
+    <xacro:include filename="$(find rover_config)/urdf/bb2.xacro" />
+    <xacro:bb2 name="loc_cam" parent_link="base_link">
+        <origin rpy="0 ${pi/6} 0" xyz="${chassis_x/2} 0.0 ${chassis_z/2 + 0.2}"/>
+    </xacro:bb2>
+  </xacro:if>
   <xacro:include filename="$(find rover_config)/urdf/vlp_16.xacro"/>
   <xacro:lidar parent_link="base_link">

Commit message: changed sensor options to arguments, fixed PTU and bb2 parameters (added coordinate Systems to SLDWORKS model), updated rviz file.

File: urdf/bb2.xacro (robot description, xacro)
@@ -10,7 +10,7 @@
     <xacro:property name="link_cam_z" value="0.036" />
     <xacro:property name="link_cam_rot_r" value="${-pi/2}" />
-    <xacro:property name="link_cam_pos_x" value="0.0" />
-    <xacro:property name="link_cam_pos_y" value="0.01625" />
-    <xacro:property name="link_cam_pos_z" value="0.0" />
+    <xacro:property name="link_cam_pos_x" value="-0.0034" />
+    <xacro:property name="link_cam_pos_y" value="0.0" />
+    <xacro:property name="link_cam_pos_z" value="${link_cam_z/2}" />
     <!-- CAMERA JOINT-->
     <joint name="joint_${name}" type="fixed">

File: urdf/marta.xacro (robot description, xacro)
@@ -2,9 +2,14 @@
 <robot name="marta" xmlns:xacro="http://www.ros.org/wiki/xacro">
   <!-- SENSOR CONFIGURATION -->
-  <xacro:property name="use_lidar"    value="true" />
-  <xacro:property name="use_imu"      value="true" />
-  <xacro:property name="use_gnss"     value="true" />
-  <xacro:property name="use_ptu"      value="true" />
-  <xacro:property name="use_loc_cam"  value="true" />
+  <xacro:arg name="use_lidar"    default="true" />
+  <xacro:arg name="use_imu"      default="true" />
+  <xacro:arg name="use_gnss"     default="true" />
+  <xacro:arg name="use_ptu"      default="true" />
+  <xacro:arg name="use_loc_cam"  default="true" />
+  <xacro:property name="use_lidar"    value="$(arg use_lidar)" />
+  <xacro:property name="use_imu"      value="$(arg use_imu)" />
+  <xacro:property name="use_gnss"     value="$(arg use_gnss)" />
+  <xacro:property name="use_ptu"      value="$(arg use_ptu)" />
+  <xacro:property name="use_loc_cam"  value="$(arg use_loc_cam)" />
   <!-- PHYSICS -->
   <xacro:property name="damping" value="2" />
@@ -363,5 +368,5 @@
     <xacro:include filename="$(find rover_config)/urdf/ptu.xacro" />
     <xacro:ptu parent_link="base_link">
-      <origin xyz="0.25 0.0 0.0" rpy="0.0 0.0 0.0"/>
+      <origin xyz="0.187 0.0 0.0" rpy="0.0 0.0 0.0"/>
     </xacro:ptu>
   </xacro:if>

File: urdf/ptu.xacro (robot description, xacro)
@@ -29,5 +29,6 @@
     <xacro:property name="tilt_lower" value="-1.57" />
     <xacro:property name="tilt_upper" value="1.57" />
-    <xacro:property name="joint_tilt_pos_z" value="0.0265" />
+    <xacro:property name="joint_tilt_pos_y" value="-0.0095" />
+    <xacro:property name="joint_tilt_pos_z" value="0.0295" />
     <xacro:property name="joint_tilt_rot_x" value="${pi/2}" />
     <!-- TILT LINK -->
@@ -37,8 +38,9 @@
     <xacro:property name="link_tilt_z" value="0.072" />
     <xacro:property name="link_tilt_pos_x" value="0.0" />
-    <xacro:property name="link_tilt_pos_y" value="0.01625" />
-    <xacro:property name="link_tilt_pos_z" value="0.0" />
+    <xacro:property name="link_tilt_pos_y" value="${0.01625 - link_tilt_y}" />
+    <xacro:property name="link_tilt_pos_z" value="${joint_tilt_pos_y}" />
     <!-- CAM JOINT -->
-    <xacro:property name="joint_cam_pos_y" value="0.036" />
+    <xacro:property name="joint_cam_pos_y" value="0.015" />
+    <xacro:property name="joint_cam_pos_z" value="${joint_tilt_pos_y}" />
     <xacro:property name="joint_cam_rot_r" value="${-pi/2}" />
     <!-- MAST JOINT -->
@@ -124,5 +126,5 @@
       <parent link="link_pan"/>
       <child link="link_tilt"/>
-      <origin xyz="0 0 ${joint_tilt_pos_z}" rpy="${joint_tilt_rot_x} 0.0 0.0"/>
+      <origin xyz="0.0 ${joint_tilt_pos_y} ${joint_tilt_pos_z}" rpy="${joint_tilt_rot_x} 0.0 0.0"/>
       <limit effort="${max_effort}" lower="${tilt_lower}" upper="${tilt_upper}" velocity="${max_velocity}"/>
       <axis xyz="0 0 1"/>
@@ -159,5 +161,5 @@
     <xacro:include filename="$(find rover_config)/urdf/bb2.xacro" />
     <xacro:bb2 name="nav_cam" parent_link="link_tilt">
-        <origin rpy="${joint_cam_rot_r} 0 0" xyz="0.0 ${joint_cam_pos_y} 0.0"/>
+        <origin rpy="${joint_cam_rot_r} 0 0" xyz="0.0 ${joint_cam_pos_y} ${joint_cam_pos_z}"/>
     </xacro:bb2>
   </xacro:macro>

Commit message: Update gazebo/rviz config for stereocam support
- Use multicam feature of gazebo camera plugin
- Define camera_frame link to follow image
  frame convention
- Set image topic in rviz to "Best Effort"
- Add stereo point cloud to rviz

File: urdf/bb2.xacro (robot description, xacro)
@@ -18,5 +18,4 @@
         <child link="link_${name}"/>
         <xacro:insert_block name="origin_cam" />
-        <axis xyz="1 0 0" />
     </joint>
     <!-- CAMERA LINK -->
@@ -45,4 +44,12 @@
       </visual>
     </link>
+    <!-- By convention the image frames axes are defines as: x-right, y-down, z-out of image  -->
+    <!-- That's why a another link for the image frame is needed. -->
+    <joint name="joint_${name}_frame" type="fixed">
+      <origin xyz="0.0 0.0 0.0" rpy="${-pi/2} 0 ${-pi/2}"/>
+      <parent link="link_${name}"/>
+      <child link="link_${name}_frame"/>
+    </joint>
+    <link name="link_${name}_frame"/>
   </xacro:macro>
 </robot>

Commit message: Fix position of optical camera frame

File: urdf/bb2.xacro (robot description, xacro)
@@ -3,5 +3,7 @@
   <xacro:macro name="bb2" params="name parent_link *origin_cam">
     <xacro:include filename="$(find rover_config)/urdf/bb2.gazebo" />
-    <xacro:sensors cam_name="${name}"/>
+    <!-- baseline defines the distance between the two optical sensors -->
+    <xacro:property name="baseline" value="0.12" />
+    <xacro:sensors cam_name="${name}" baseline="${baseline}"/>
     <!-- PARAMETERS -->
     <xacro:property name="link_cam_mass" value="1.0" />
@@ -47,5 +49,5 @@
     <!-- That's why a another link for the image frame is needed. -->
     <joint name="joint_${name}_frame" type="fixed">
-      <origin xyz="0.0 0.0 0.0" rpy="${-pi/2} 0 ${-pi/2}"/>
+      <origin xyz="0.0 ${baseline/2} 0.018" rpy="${-pi/2} 0 ${-pi/2}"/>
       <parent link="link_${name}"/>
       <child link="link_${name}_frame"/>
